File: lab3/Schematic/Schematic.kicad_sch (KiCad schematic)
At the start: 24 parts, among them J1 Raspberry_Pi_4, J2 Conn_01x06_Pin, J3 Conn_01x06_Pin, J4 Conn_01x13_Socket, M1 Motor_Servo, U1 MCP2515-xST, U2 L298N, U3 STM32F401RETx, U4 ACS712xLCTR-05B, U5 ACS712xLCTR-05B, U6 ACS712xLCTR-05B, U7 STM32F401RETx, U8 SN65HVD230

Commit message: First draft of pinout for CAN lab
Parts:
- added J5: Raspberry_Pi_4, symbol Connector:Raspberry_Pi_4
Connections:
- net Z2_INT_CAN_A: now reaches U7.29 (PB10)
- net Z2_INT_CAN_A: now also U1.13 (~{INT})
- net Z2_INT_CAN_B: now reaches U7.41 (PA8)
- net Z2_SCLK: now reaches U7.55 (PB3)
- net Z2_MISO: now reaches U7.56 (PB4)
- net Z2_MOSI: now reaches U7.57 (PB5)
- net Z2_CS_CAN_A: now reaches U7.58 (PB6)
- net Z1_SCLK: now reaches U1.14 (SCK)
- net Z1_SCLK: now also J5.23 (SCLK_SPI0/GPIO11)
- net Z1_MOSI: now reaches U1.16 (SI)
- net Z1_MOSI: now also J5.19 (MOSI_SPI0/GPIO10)
- net Z1_MISO: now reaches U1.17 (SO)
- net Z1_MISO: now also J5.21 (MISO_SPI0/GPIO09)
- net Z1_CS_CAN_A: now reaches U1.18 (~{CS})
- net Z1_CS_CAN_A: now also J5.24 (~{CE0}_SPI0/GPIO08)
- net Z3_INT_CAN_A: now reaches U3.29 (PB10)
- net Z3_CS_CAN_B: now reaches U3.38 (PC7)
- net Z3_INT_CAN_B: now reaches U3.41 (PA8)
- net Z3_SCLK: now reaches U3.55 (PB3)
- net Z3_MISO: now reaches U3.56 (PB4)
- net Z3_MOSI: now reaches U3.57 (PB5)
- net Z3_CS_CAN_A: now reaches U3.58 (PB6)
- new net: J5.1 (3V3), J5.17 (3V3)
- new net: J5.14 (GND), J5.20 (GND), J5.25 (GND), J5.30 (GND), J5.34 (GND), J5.39 (GND), J5.6 (GND), J5.9 (GND)
- new net: J5.2 (5V), J5.4 (5V)
- new net Z1_CS_CAN_B: J5.26 (~{CE1}_SPI0/GPIO07)
- new net Z1_INT_CAN_A: J5.18 (GPIO24/SDIO_DAT0)
- new net Z1_INT_CAN_B: J5.22 (GPIO25/SDIO_DAT1)
Other:
- note added: "Control (Zone 1)"
- note added: "Drivetrain (Zone 3)"
- note added: "Steering (Zone 2)"
- moved on the sheet: C1, U1, U3, U8

Commit message: Schematic tenativley complete for CAN lab
Parts:
- removed A1: Arduino_UNO_R3, Module:Arduino_UNO_R3, symbol MCU_Module:Arduino_UNO_R3
- removed D1: LED G, symbol Device:LED
- removed D2: LED Y, symbol Device:LED
- removed D3: LED R, symbol Device:LED
- removed D4: LED B, symbol Device:LED
- removed J1: Raspberry_Pi_4, symbol Connector:Raspberry_Pi_4
- removed J2, J3: Conn_01x06_Pin, LED_THT:LED_D5.0mm_IRGrey, symbol Connector:Conn_01x06_Pin
- removed J4: Conn_01x13_Socket, symbol Connector:Conn_01x13_Socket
- removed M1: Motor_Servo, Package_DIP:DIP-16_W7.62mm, symbol Motor:Motor_Servo
- removed R10, R7, R8, R9: 470, Package_DIP:DIP-8_W7.62mm, symbol Device:R
- removed R11: 10K, Package_DIP:DIP-8_W7.62mm, symbol Device:R
- removed U2: L298N, Package_TO_SOT_THT:TO-220-15_P2.54x5.08mm_StaggerOdd_Lead4.58mm_Vertical, symbol Driver_Motor:L298N
- removed U4, U5, U6: ACS712xLCTR-05B, Package_SO:SOIC-8_3.9x4.9mm_P1.27mm, symbol Sensor_Current:ACS712xLCTR-05B
- added C10, C13, C14, C17, C18, C2, C21, C22, C3, C5, C6, C9: 22pF, Capacitor_SMD:C_0603_1608Metric, symbol Device:C
- added C11, C15, C19, C23, C4, C7: 100nF, symbol Device:C
- added C12, C16, C20, C24, C8: 100nF, Capacitor_SMD:C_0603_1608Metric, symbol Device:C
- added D10, D14, D15, D19, D20, D9: LED R, symbol Device:LED
- added D11, D12, D13, D16, D17, D18, D23: LED G, symbol Device:LED
- added J10: Zone 3 (Rear) Test Point Breakout, symbol Connector:Conn_01x13_Socket
- added J6: Zone 1 (PI) Test Point Breakout, symbol Connector:Conn_01x13_Socket
- added J7, J8: Conn_01x06_Pin, LED_THT:LED_D5.0mm_IRGrey, symbol Connector:Conn_01x06_Pin
- added J9: Zone 2 (Front) Test Point Breakout, symbol Connector:Conn_01x13_Socket
- added JP1, JP10, JP11, JP12, JP13, JP14, JP15, JP16, JP17, JP18, JP19, JP2, JP20, JP3, JP4, JP5, JP6, JP7, JP8, JP9: (no value), symbol Jumper:Jumper_2_Bridged
- added M2: Motor_Servo, Package_DIP:DIP-16_W7.62mm, symbol Motor:Motor_Servo
- added R1, R12, R14, R16, R3, R5: 10k, Resistor_SMD:R_0603_1608Metric, symbol Device:R
- added R13, R15, R17, R2, R4, R6: 47K, Resistor_SMD:R_0603_1608Metric, symbol Device:R
- added R18, R19, R20, R21: 120, Resistor_SMD:R_0603_1608Metric, symbol Device:R
- added R25, R26, R27, R28, R29, R30, R31, R32, R33, R34, R35, R36, R39: 560, Package_DIP:DIP-8_W7.62mm, symbol Device:R
- added TP1: UDP_RX, TestPoint:TestPoint_Keystone_5015_Micro_Mini, symbol Connector:TestPoint
- added TP13: MOTOR_DIR, TestPoint:TestPoint_Keystone_5015_Micro_Mini, symbol Connector:TestPoint
- added TP14: PWM_SET, TestPoint:TestPoint_Keystone_5015_Micro_Mini, symbol Connector:TestPoint
- added TP15: MOTOR_PWM_OUT, TestPoint:TestPoint_Keystone_5015_Micro_Mini, symbol Connector:TestPoint
- added TP16: Z3_CAN_TX_A, TestPoint:TestPoint_Keystone_5015_Micro_Mini, symbol Connector:TestPoint
- added TP17: Z3_CAN_TX_B, TestPoint:TestPoint_Keystone_5015_Micro_Mini, symbol Connector:TestPoint
- added TP18: Z3_CAN_RX_A, TestPoint:TestPoint_Keystone_5015_Micro_Mini, symbol Connector:TestPoint
- added TP19: Z3_CAN_RX_B, TestPoint:TestPoint_Keystone_5015_Micro_Mini, symbol Connector:TestPoint
- added TP2, Z2_CAN_TX_A: CMD_TX, TestPoint:TestPoint_Keystone_5015_Micro_Mini, symbol Connector:TestPoint
- added TP3: CAN_TX_A, TestPoint:TestPoint_Keystone_5015_Micro_Mini, symbol Connector:TestPoint
- added TP4: CAN_TX_B, TestPoint:TestPoint_Keystone_5015_Micro_Mini, symbol Connector:TestPoint
- added TP6, TP8: Z2_CAN_RX_B, TestPoint:TestPoint_Keystone_5015_Micro_Mini, symbol Connector:TestPoint
- added TP7: Z2_CAN_RX_A, TestPoint:TestPoint_Keystone_5015_Micro_Mini, symbol Connector:TestPoint
- added TP9: Z2_RELAY_TX, TestPoint:TestPoint_Keystone_5015_Micro_Mini, symbol Connector:TestPoint
- added U10, U12, U14, U16, U18: SN65HVD230, Package_SO:SOIC-8_3.9x4.9mm_P1.27mm, symbol Interface_CAN_LIN:SN65HVD230
- added U11, U13, U15, U17, U9: MCP2515-xST, Package_SO:TSSOP-20_4.4x6.5mm_P0.65mm, symbol Interface_CAN_LIN:MCP2515-xST
- added U20: L298N, Package_TO_SOT_THT:TO-220-15_P2.54x5.08mm_StaggerOdd_Lead4.58mm_Vertical, symbol Driver_Motor:L298N
- added Y1, Y2, Y3, Y4, Y5, Y6: CX3225SB16000H0FLJCC, CX3225SB16000H0FLJCC:OSCCC320X250X60N, symbol Device:CX3225SB16000H0FLJCC
Connections:
- net +12V: now also U20.9 (Vss)
- net +3.3V: now also U1.20 (VDD), C11.1, C12.1, C15.1, C16.1, C19.1, C20.1, C23.1, C24.1, C4.1, C7.1, C8.1, R1.1, R12.1, R14.1, R16.1, R3.1, R5.1, U10.3 (VCC), U11.20 (VDD), U12.3 (VCC), U13.20 (VDD), U14.3 (VCC), U15.20 (VDD), U16.3 (VCC), U17.20 (VDD), U18.3 (VCC), U9.20 (VDD)
- net +5V: now also J7.2 (Pin_2), J8.2 (Pin_2), M2.2 (+), U20.4 (Vs)
- net CANH_A_Z1: now also JP3.1 (A)
- net CANL_A_Z1: now also JP4.2 (B)
- net DIR_A: now also U3.61 (PB8), J10.11 (Pin_11)
- net GND: now also J5.14 (GND), J5.20 (GND), J5.25 (GND), J5.30 (GND), J5.34 (GND), J5.39 (GND), J5.6 (GND), J5.9 (GND), C10.2, C11.2, C12.2, C13.2, C14.2, C15.2, C16.2, C17.2, C18.2, C19.2, C2.2, C20.2, C21.2, C22.2, C23.2, C24.2, C3.2, C4.2, C5.2, C6.2, C7.2, C8.2, C9.2, D10.1 (K), D11.1 (K), D12.1 (K), D13.1 (K), D14.1 (K), D15.1 (K), D16.1 (K), D17.1 (K), D18.1 (K), D19.1 (K), D20.1 (K), D23.1 (K), D9.1 (K), J10.1 (Pin_1), J10.2 (Pin_2), J6.1 (Pin_1), J6.2 (Pin_2), J7.5 (Pin_5), J8.5 (Pin_5), J9.1 (Pin_1), J9.2 (Pin_2), M2.3 (-), R13.2, R15.2, R17.2, R2.2, R4.2, R6.2, U10.2 (GND), U11.10 (VSS), U12.2 (GND), U13.10 (VSS), U14.2 (GND), U15.10 (VSS), U16.2 (GND), U17.10 (VSS), U18.2 (GND), U20.8 (GND), U9.10 (VSS), Y1.2 (GND), Y1.4 (GND), Y2.2 (GND), Y2.4 (GND), Y3.2 (GND), Y3.4 (GND), Y4.2 (GND), Y4.4 (GND), Y5.2 (GND), Y5.4 (GND), Y6.2 (GND), Y6.4 (GND)
- net PWM_SET: now also U3.9 (PC1), J10.9 (Pin_9), TP14.1
- net UDP_RX: now also J5.3 (SDA_I2C1/GPIO02), J6.3 (Pin_3), TP1.1
- net Z1_CS_CAN_B: now also U13.18 (~{CS})
- net Z1_INT_CAN_A: now also U1.13 (~{INT})
- net Z1_INT_CAN_B: now also U13.13 (~{INT})
- net Z1_MISO: now also U13.17 (SO)
- net Z1_MOSI: now also U13.16 (SI)
- net Z1_SCLK: now also U13.14 (SCK)
- net Z2_CS_CAN_A: now also U9.18 (~{CS})
- net Z2_CS_CAN_B: now also U7.38 (PC7), U15.18 (~{CS})
- net Z2_INT_CAN_A: now also U9.13 (~{INT}); no longer U1.13 (~{INT})
- net Z2_INT_CAN_B: now also U15.13 (~{INT})
- net Z2_MISO: now also U15.17 (SO), U9.17 (SO)
- net Z2_MOSI: now also U15.16 (SI), U9.16 (SI)
- net Z2_SCLK: now also U15.14 (SCK), U9.14 (SCK)
- net Z3_CS_CAN_A: now also U11.18 (~{CS})
- net Z3_CS_CAN_B: now also U17.18 (~{CS})
- net Z3_INT_CAN_A: now also U11.13 (~{INT})
- net Z3_INT_CAN_B: now also U17.13 (~{INT})
- net Z3_MISO: now also U11.17 (SO), U17.17 (SO)
- net Z3_MOSI: now also U11.16 (SI), U17.16 (SI)
- net Z3_SCLK: now also U11.14 (SCK), U17.14 (SCK)
- net at U8.5 (Vref): now also R2.1
- net SERVO_PWM: now reaches U7.14 (PA0)
- net SERVO_PWM: now also J9.9 (Pin_9), M2.1 (PWM)
- net Z2_DEG_A: now reaches U7.15 (PA1)
- net Z2_DEG_A: now also J9.7 (Pin_7), R25.2
- net Z2_TEST_BUTTON: now reaches U7.2 (PC13)
- net Z2_TEST_BUTTON: now also U3.2 (PC13)
- net Z2_DEG_B: now reaches U7.20 (PA4)
- net Z2_DEG_B: now also J9.8 (Pin_8), R26.2
- net FR_BLINK: now reaches U7.22 (PA6)
- net FR_BLINK: now also J9.11 (Pin_11), R28.2
- net Z2_CAN_TX_A: now reaches U7.23 (PA7)
- net Z2_CAN_TX_A: now also J9.5 (Pin_5), Z2_CAN_TX_A.1
- net Z2_ERR: now reaches U7.26 (PB0)
- net Z2_ERR: now also J9.13 (Pin_13), R29.2
- net Z2_CAN_RX_B: now reaches U7.42 (PA9)
- net Z2_CAN_RX_B: now also J9.4 (Pin_4), TP6.1
- net Z2_CAN_RX_A: now reaches U7.43 (PA10)
- net Z2_CAN_RX_A: now also J9.3 (Pin_3), TP7.1
- net Z2_CAN_TX_B: now reaches U7.61 (PB8)
- net Z2_CAN_TX_B: now also J9.6 (Pin_6), TP8.1
- net FL_BLINK: now reaches U7.62 (PB9)
- net FL_BLINK: now also J9.10 (Pin_10), R27.2
- net Z2_RELAY_TX: now reaches U7.9 (PC1)
- net Z2_RELAY_TX: now also J9.12 (Pin_12), TP9.1
- net at U1.19 (~{RESET}): now also R1.2
- net at U1.8 (OSC2): now also C2.1, Y1.1
- net at U1.9 (OSC1): now also C3.1, Y1.3
- net ENC_LEFT_B: now reaches U3.14 (PA0)
- net ENC_LEFT_B: now also J7.4 (Pin_4), J8.4 (Pin_4)
- net ENC_RIGHT_A: now reaches U3.15 (PA1)
- net ENC_RIGHT_A: now also J7.3 (Pin_3)
- net ENC_RIGHT_B: now reaches U3.20 (PA4)
- net RL_BLINK: now reaches U3.22 (PA6)
- net RL_BLINK: now also J10.12 (Pin_12), R32.2
- net MOTOR_LEFT_PWM: now reaches U3.23 (PA7)
- net MOTOR_LEFT_PWM: now also U20.10 (IN3)
- net Z3_CAN_TX_B: now reaches U3.25 (PC5)
- net Z3_CAN_TX_B: now also J10.6 (Pin_6), TP17.1
- net MOTOR_RIGHT_DIR: now reaches U3.26 (PB0)
- net MOTOR_RIGHT_DIR: now also U20.7 (IN2)
- net Z3_CAN_TX_A: now reaches U3.37 (PC6)
- net Z3_CAN_TX_A: now also J10.5 (Pin_5), TP16.1
- net Z3_CAN_RX_B: now reaches U3.39 (PC8)
- net Z3_CAN_RX_B: now also J10.4 (Pin_4), TP19.1
- net Z3_CAN_RX_A: now reaches U3.40 (PC9)
- net Z3_CAN_RX_A: now also J10.3 (Pin_3), TP18.1
- net ENC_LEFT_A: now reaches U3.42 (PA9)
- net ENC_LEFT_A: now also J8.3 (Pin_3)
- net MOTOR_RIGHT_PWM: now reaches U3.43 (PA10)
- net MOTOR_RIGHT_PWM: now also TP15.1, U20.5 (IN1)
- net Z3_DEG_A: now reaches U3.51 (PC10)
- net Z3_DEG_A: now also J10.7 (Pin_7), R30.2
- net Z3_DEG_B: now reaches U3.52 (PC11)
- net Z3_DEG_B: now also J10.8 (Pin_8), R31.2
- net Z3_ERR: now reaches U3.53 (PC12)
- net Z3_ERR: now also R34.2
- net RR_BLINK: now reaches U3.62 (PB9)
- net RR_BLINK: now also J10.13 (Pin_13), R33.2
- net MOTOR_LEFT_DIR: now reaches U3.8 (PC0)
- net MOTOR_LEFT_DIR: now also TP13.1, U20.12 (IN4)
- net Z1_CAN_TX_A: now reaches J5.29 (GPCLK1/GPIO05)
- net Z1_CAN_TX_A: now also J6.5 (Pin_5), J6.6 (Pin_6), TP3.1
- net Z1_CAN_TX_B: now reaches J5.31 (GPCLK2/GPIO06)
- net Z1_CAN_TX_B: now also TP4.1
- net Z1_DEG_A: now reaches J5.33 (GPIO13/PWM1)
- net Z1_DEG_A: now also J6.7 (Pin_7), R35.2
- net Z1_DEG_B: now reaches J5.35 (GPIO19/SPI1_MISO/PCM_FS)
- net Z1_DEG_B: now also J6.8 (Pin_8), R36.2
- net Z1_ERR: now reaches J5.37 (GPIO26/SDIO_DAT2)
- net Z1_ERR: now also R39.2
- net Z1_CMD_TX: now reaches J5.5 (SCL_I2C1/GPIO03)
- net Z1_CMD_TX: now also TP2.1
- new net: D17.2 (A), R33.1
- new net: R4.1, U10.5 (Vref)
- new net: C6.1, U9.9 (OSC1), Y2.3
- new net: D23.2 (A), R39.1
- new net: C10.1, U11.9 (OSC1), Y3.3
- new net: C14.1, U13.9 (OSC1), Y4.3
- new net: JP1.1 (A), R18.1
- new net: D19.2 (A), R35.1
- new net: D10.2 (A), R26.1
- new net: JP2.1 (A), R18.2
- new net: U11.1 (TXCAN), U12.1 (D)
- new net: R5.2, U11.19 (~{RESET})
- new net: U11.2 (RXCAN), U12.4 (R)
- new net: C9.1, U11.8 (OSC2), Y3.1
- new net: D11.2 (A), R27.1
- new net: JP10.2 (B), R19.2
- new net: D16.2 (A), R32.1
- new net: D13.2 (A), R29.1
- new net: D14.2 (A), R30.1
- new net: R15.1, U16.5 (Vref)
- new net: U17.1 (TXCAN), U18.1 (D)
- new net: R16.2, U17.19 (~{RESET})
- new net: U17.2 (RXCAN), U18.4 (R)
- new net: C21.1, U17.8 (OSC2), Y6.1
- new net: C22.1, U17.9 (OSC1), Y6.3
- new net: D18.2 (A), R34.1
- new net: R12.2, U13.19 (~{RESET})
- new net: JP11.1 (A), R20.1
- new net: C17.1, U15.8 (OSC2), Y5.1
- new net: C18.1, U15.9 (OSC1), Y5.3
- new net: R3.2, U9.19 (~{RESET})
- new net: D20.2 (A), R36.1
- new net: JP9.2 (B), R19.1
- new net: JP20.2 (B), R21.2
- new net: D15.2 (A), R31.1
- new net: C13.1, U13.8 (OSC2), Y4.1
- new net: R14.2, U15.19 (~{RESET})
- new net: U13.1 (TXCAN), U14.1 (D)
- new net: U13.2 (RXCAN), U14.4 (R)
- new net: R6.1, U12.5 (Vref)
- new net: R17.1, U18.5 (Vref)
- new net: D12.2 (A), R28.1
- new net: D9.2 (A), R25.1
- new net: U15.1 (TXCAN), U16.1 (D)
- new net: U15.2 (RXCAN), U16.4 (R)
- new net: C5.1, U9.8 (OSC2), Y2.1
- new net: J7.1 (Pin_1), U20.2 (OUT1)
- new net: J7.6 (Pin_6), U20.3 (OUT2)
- new net: R13.1, U14.5 (Vref)
- new net: JP19.2 (B), R21.1
- new net: JP12.1 (A), R20.2
- new net: U10.1 (D), U9.1 (TXCAN)
- new net: U10.4 (R), U9.2 (RXCAN)
- new net: J8.1 (Pin_1), U20.13 (OUT3)
- new net: J8.6 (Pin_6), U20.14 (OUT4)
- new net CANH_A: JP1.2 (B), JP3.2 (B), JP5.2 (B), JP7.2 (B), JP9.1 (A)
- new net CANH_A_Z2: JP5.1 (A), U10.7 (CANH)
- new net CANH_A_Z3: JP7.1 (A), U12.7 (CANH)
- new net CANH_B: JP11.2 (B), JP13.2 (B), JP15.2 (B), JP17.2 (B), JP19.1 (A)
- new net CANH_B_Z1: JP13.1 (A), U14.7 (CANH)
- new net CANH_B_Z2: JP15.1 (A), U16.7 (CANH)
- new net CANH_B_Z3: JP17.1 (A), U18.7 (CANH)
- new net CANL_A: JP10.1 (A), JP2.2 (B), JP4.1 (A), JP6.1 (A), JP8.1 (A)
- new net CANL_A_Z2: JP6.2 (B), U10.6 (CANL)
- new net CANL_A_Z3: JP8.2 (B), U12.6 (CANL)
- new net CANL_B: JP12.2 (B), JP14.1 (A), JP16.1 (A), JP18.1 (A), JP20.1 (A)
- new net CANL_B_Z1: JP14.2 (B), U14.6 (CANL)
- new net CANL_B_Z2: JP16.2 (B), U16.6 (CANL)
- new net CANL_B_Z3: JP18.2 (B), U18.6 (CANL)
- new net PWM_OUT: J10.10 (Pin_10)
- new net Z1_CMD_RX: J6.4 (Pin_4)
- new net _: J6.10 (Pin_10), J6.11 (Pin_11), J6.12 (Pin_12), J6.13 (Pin_13), J6.9 (Pin_9)
Other:
- note added: "CAN controller schematic copied from: https://wiki.seeedstudio.com/xiao-can-bus-expansion"
- note added: "Schematic is currently missing: - Everything to do with power - All of the oscilators and support for STM 32 processors - Remember to have a way to flash - All of the current sensing - Fun things - Pixels - Speaker"
- note removed: "Pin D14 Pin D15"
- moved on the sheet: C1, J5, U1, U3, U7, U8

Commit message: Schematic 1.0
Other:
- title: (none) -> CAN Lab Scheumatic 
Changed lines of the file:
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@@
 	(generator_version "10.0")
 	(paper "C")
+	(title_block
+		(title "CAN Lab Scheumatic ")
+		(date "2026-10-22")
+	)
 	(text "Right Motor"
 		(exclude_from_sim no)
