File: lab4/Schematic/Schematic.kicad_pcb (KiCad board)
At the start: 2 copper layers, 319 parts, among them IC1 TPS564252DRLR, IC2 TPS564252DRLR, IC3 TPS564252DRLR, IC4 TPS564252DRLR, IC5 TPS564252DRLR, IC6 TPS564252DRLR, J1 XT60-M, J10 CANA_Z1, J11 CANA_Z1, J12 CANA_Z1, J13 CANA_Z1, J14 CANA_Z1, J15 CANA_Z1, J2 Z2_SWD, J3 Z2_SWD, J4 Z3_USART, J5 Raspberry_Pi_4, J6 Z3_USART, J7 MOTOR_RIGHT, J8 MOTOR_LEFT, J9 SERVO, Q2 IRF4905, U1 MCP2515-xST, U10 SN65HVD230, U11 MCP2515-xST, U12 SN65HVD230, U13 MCP2515-xST, U14 SN65HVD230, U15 MCP2515-xST, U16 SN65HVD230, U17 MCP2515-xST, U18 SN65HVD230, U2 ACS712xLCTR-05B, U20 L298N, U3 STM32F401RETx, U4 ACS712xLCTR-05B, U5 INA181, U7 STM32F401RETx, U8 SN65HVD230, U9 MCP2515-xST, Y1 CX3225SB16000H0FLJCC, Y2 CX3225SB16000H0FLJCC, Y3 CX3225SB16000H0FLJCC, Y4 CX3225SB16000H0FLJCC, Y5 CX3225SB16000H0FLJCC, Y6 CX3225SB16000H0FLJCC, Y7 ABS25-32.768KHZ-6-T, Y8 ABS25-32.768KHZ-6-T

Commit message: Schematic Updates
Parts:
- removed F1: 15 A, Resistor_THT:R_Axial_DIN0922_L20.0mm_D9.0mm_P25.40mm_Horizontal
- removed L1, L2, L3: 2.2uH, Inductor_SMD:L_Eaton_SDCHA1V80
- added C86: 470 uF, Capacitor_THT:CP_Radial_D8.0mm_P3.80mm, F.Cu at (84.2, -282.0)
- added C87: 0.1uF, Capacitor_SMD:C_0603_1608Metric, F.Cu at (366.8, -64.5)
- added D28: D_Schottky, Diode_SMD:D_SMB, F.Cu at (191.4, -386.1)
- added D29: D_Schottky, Diode_SMD:D_SMB, F.Cu at (191.4, -380.6)
- added D30: D_Schottky, Diode_SMD:D_SMB, F.Cu at (191.4, -375.1)
- added D31: D_Schottky, Diode_SMD:D_SMB, F.Cu at (191.4, -369.5)
- added D32: D_Schottky, Diode_SMD:D_SMB, F.Cu at (191.4, -363.9)
- added D33: D_Schottky, Diode_SMD:D_SMB, F.Cu at (191.4, -358.4)
- added D34: D_Schottky, Diode_SMD:D_SMB, F.Cu at (191.4, -352.9)
- added D35: D_Schottky, Diode_SMD:D_SMB, F.Cu at (191.4, -347.3)
- added D36: POWER, LED_SMD:LED_0603_1608Metric, F.Cu at (390.8, -76.0)
- added D37: POWER, LED_SMD:LED_0603_1608Metric, F.Cu at (88.9, 107.3)
- added D38: POWER, LED_SMD:LED_0603_1608Metric, F.Cu at (107.5, -298.8)
- added D39: POWER, LED_SMD:LED_0603_1608Metric, F.Cu at (107.3, -326.9)
- added D40: POWER, LED_SMD:LED_0603_1608Metric, F.Cu at (232.5, 105.3)
- added D41: POWER, LED_SMD:LED_0603_1608Metric, F.Cu at (421.5, -59.5)
- added D42: POWER, LED_SMD:LED_0603_1608Metric, F.Cu at (-106.3, -151.5)
- added D43: RXCAN, LED_SMD:LED_0603_1608Metric, F.Cu at (432.6, -96.5)
- added D44: TXCAN, LED_SMD:LED_0603_1608Metric, F.Cu at (438.1, -83.0)
- added D45: RXCAN, LED_SMD:LED_0603_1608Metric, F.Cu at (275.3, 121.1)
- added D46: TXCAN, LED_SMD:LED_0603_1608Metric, F.Cu at (275.3, 123.7)
- added D47: RXCAN, LED_SMD:LED_0603_1608Metric, F.Cu at (279.4, 113.4)
- added D48: TXCAN, LED_SMD:LED_0603_1608Metric, F.Cu at (279.4, 116.0)
- added D49: RXCAN, LED_SMD:LED_0603_1608Metric, F.Cu at (279.4, 118.6)
- added D50: TXCAN, LED_SMD:LED_0603_1608Metric, F.Cu at (279.4, 121.1)
- added D51: RXCAN, LED_SMD:LED_0603_1608Metric, F.Cu at (279.4, 123.7)
- added D52: TXCAN, LED_SMD:LED_0603_1608Metric, F.Cu at (283.4, 113.4)
- added D53: RXCAN, LED_SMD:LED_0603_1608Metric, F.Cu at (283.4, 116.0)
- added D54: TXCAN, LED_SMD:LED_0603_1608Metric, F.Cu at (283.4, 118.6)
- added F2: 3557-2, 3557_2:FUSE_3557-2, F.Cu at (-124.1, -182.6)
- added L7: 4.7uH, Inductor_SMD:L_Eaton_SDCHA1V80, F.Cu at (424.0, -65.0)
- added L8: 4.7uH, Inductor_SMD:L_Eaton_SDCHA1V80, F.Cu at (235.0, 99.8)
- added L9: 4.7uH, Inductor_SMD:L_Eaton_SDCHA1V80, F.Cu at (109.8, -332.4)
- added R75: 91K, Resistor_SMD:R_0603_1608Metric, F.Cu at (106.5, 106.2)
- added R78: 4K7, Resistor_SMD:R_0603_1608Metric, F.Cu at (369.1, -68.3)
- added R79: 120, Resistor_SMD:R_0603_1608Metric, F.Cu at (363.3, -64.5)
- added R80: 1K, Resistor_SMD:R_0603_1608Metric, F.Cu at (390.8, -80.0)
- added R81: 1K, Resistor_SMD:R_0603_1608Metric, F.Cu at (88.9, 103.3)
- added R82: 1K, Resistor_SMD:R_0603_1608Metric, F.Cu at (107.5, -302.8)
- added R83: 470, Resistor_SMD:R_0603_1608Metric, F.Cu at (107.3, -330.9)
- added R84: 470, Resistor_SMD:R_0603_1608Metric, F.Cu at (232.5, 101.3)
- added R85: 470, Resistor_SMD:R_0603_1608Metric, F.Cu at (421.5, -63.5)
- added R86: 1K, Resistor_SMD:R_0603_1608Metric, F.Cu at (-102.3, -152.0)
- added R87: 470, Resistor_SMD:R_0603_1608Metric, F.Cu at (436.5, -96.5)
- added R88: 470, Resistor_SMD:R_0603_1608Metric, F.Cu at (435.0, -83.0)
- added R89: 470, Resistor_SMD:R_0603_1608Metric, F.Cu at (287.4, 120.9)
- added R90: 470, Resistor_SMD:R_0603_1608Metric, F.Cu at (287.4, 123.4)
- added R91: 470, Resistor_SMD:R_0603_1608Metric, F.Cu at (291.4, 113.3)
- added R92: 470, Resistor_SMD:R_0603_1608Metric, F.Cu at (291.4, 115.8)
- added R93: 470, Resistor_SMD:R_0603_1608Metric, F.Cu at (291.4, 118.4)
- added R94: 470, Resistor_SMD:R_0603_1608Metric, F.Cu at (291.4, 120.9)
- added R95: 470, Resistor_SMD:R_0603_1608Metric, F.Cu at (291.4, 123.4)
- added R96: 470, Resistor_SMD:R_0603_1608Metric, F.Cu at (295.4, 113.3)
- added R97: 470, Resistor_SMD:R_0603_1608Metric, F.Cu at (295.4, 115.8)
- added R98: 470, Resistor_SMD:R_0603_1608Metric, F.Cu at (295.4, 118.4)
- added REF**: MODULE_RASPBERRY_PI_4B_4GB, RASPBERRY_PI_4B_4GB:MODULE_RASPBERRY_PI_4B_4GB, F.Cu at (507.4, -79.3)
- added S5: TEST, SWT0210_045026GSA:SW_SWT0210-045026GSA_REVA, F.Cu at (364.8, -70.8)
- added TP50: PG, TestPoint:TestPoint_Keystone_5015_Micro_Mini, F.Cu at (439.4, -53.0)
- added TP51: PG, TestPoint:TestPoint_Keystone_5015_Micro_Mini, F.Cu at (408.6, -69.5)
- added TP52: PG, TestPoint:TestPoint_Keystone_5015_Micro_Mini, F.Cu at (106.8, 113.8)
- added TP53: PG, TestPoint:TestPoint_Keystone_5015_Micro_Mini, F.Cu at (250.4, 111.8)
- added TP54: PG, TestPoint:TestPoint_Keystone_5015_Micro_Mini, F.Cu at (125.2, -320.4)
- added TP55: PG, TestPoint:TestPoint_Keystone_5015_Micro_Mini, F.Cu at (125.4, -292.2)
- J5: moved to B.Cu
- LS1, LS2: value PS1240P02BT -> BUZZER
- R71: value 1ohm -> 200m; footprint Resistor_THT:R_Axial_Power_L48.0mm_W12.5mm_P60.96mm -> Resistor_THT:R_Axial_DIN0516_L15.5mm_D5.0mm_P25.40mm_Horizontal
- R76: value 30k -> 10K
- TP29: value Z3_BOOT0 -> Z2_BOOT0
- TP30: value Z3_MCO -> Z2_MCO
- moved JP33 444.1 mm to (92.3, 114.6), turned to -90 degrees
- moved C84 443.9 mm to (101.7, 113.6)
- moved C83 443.5 mm to (101.7, 110.1)
- moved L6 439.0 mm to (91.4, 101.8)
- moved TP49 435.5 mm to (96.8, 113.6)
- moved C79 435.2 mm to (94.9, 96.0), turned to 90 degrees
- moved C85 432.1 mm to (101.5, 106.6)
- moved C80 430.6 mm to (96.9, 96.1), turned to 90 degrees
- moved R74 430.2 mm to (104.5, 113.1), turned to -90 degrees
- moved C82 429.8 mm to (106.5, 103.2), turned to 180 degrees
- moved C81 429.0 mm to (103.0, 98.8), turned to -90 degrees
- moved JP32 428.3 mm to (91.9, 99.3), turned to -90 degrees
- moved IC6 422.5 mm to (101.5, 103.1)
- moved R77 421.3 mm to (106.5, 109.4)
- moved R73 420.2 mm to (100.0, 98.7), turned to -90 degrees
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Connections:
- net Net-(J5-3V3-Pad1) renamed /PI_3.3V
- C62 pad 1: +3.3V_Z3 -> Net-(JP30-A)
- C70 pad 2: /Z3_NRST -> /Z2_NRST
- C72 pad 1: +3.3V_Z3 -> Net-(JP31-A)
- FB2 pad 1: +3.3V_Z3 -> +3.3V_Z2
- J5 pad 18: /Z1_INT_CAN_A -> /Z1_INT_CAN_B
- J5 pad 22: /Z1_INT_CAN_B -> /Z1_INT_CAN_A
- J7 pad 4: /ENC_LEFT_B -> /ENC_RIGHT_B
- JP25 pad 2: +3.3V_Z1 -> Net-(JP2-C)
- JP31 pad 2: +3.3V_Z3 -> +3.3V_Z2
- R66 pad 1: /Z3_BOOT0 -> /Z2_BOOT0
- R69 pad 1: +3.3V_Z3 -> +3.3V_Z2
- R71 pad 2: Net-(U5-+) -> Net-(J9-Pin_2)
- S3 pad 3: /Z3_NRST -> /Z2_NRST
- S3 pad 4: /Z3_NRST -> /Z2_NRST
- TP29 pad 1: /Z3_BOOT0 -> /Z2_BOOT0
- U20 pad 1: unconnected-(U20-SENSE_A-Pad1) -> GND
- U20 pad 11: unconnected-(U20-EnB-Pad11) -> +5V_Z3
- U20 pad 4: +5V_Z3 -> +12V
- U20 pad 6: unconnected-(U20-EnA-Pad6) -> +5V_Z3
- U20 pad 9: +12V -> +5V_Z3
- U3 pad 1: +3.3V_Z3 -> Net-(JP30-A)
- U5 pad 3: Net-(U5-+) -> +7V_Z2
- U7 pad 1: +3.3V_Z3 -> Net-(JP31-A)
- U7 pad 60: /Z3_BOOT0 -> /Z2_BOOT0
- U7 pad 7: /Z3_NRST -> /Z2_NRST
Routing:
- net /CANH_A: track 86.3 -> 10.8 mm, vias 6 -> 0
- net /CANL_A: track 70.9 -> 0.00 mm
- net GND: track 106.8 -> 161.3 mm, vias 70 -> 116
- net Net-(D39-A): track 0.00 -> 27.7 mm
- net Net-(D37-A): track 0.00 -> 27.7 mm
- net Net-(D36-A): track 0.00 -> 27.7 mm
- net Net-(D38-A): track 0.00 -> 27.7 mm
- net Net-(IC5-VIN): track 0.00 -> 21.0 mm
- net Net-(IC2-VIN): track 0.00 -> 21.0 mm
- net Net-(IC6-VIN): track 0.00 -> 21.0 mm
- net Net-(IC4-VIN): track 0.00 -> 21.0 mm
- net Net-(IC5-EN): track 0.00 -> 14.4 mm, vias 0 -> 2
- net Net-(IC2-EN): track 0.00 -> 14.4 mm, vias 0 -> 2
- net Net-(IC6-EN): track 0.00 -> 14.4 mm, vias 0 -> 2
- net Net-(IC4-EN): track 0.00 -> 14.4 mm, vias 0 -> 2
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- added copper zone on F.Cu, net Net-(D36-A)
- added copper zone on F.Cu, net Net-(D37-A)
- added copper zone on F.Cu, net Net-(D38-A)
- added copper zone on F.Cu, net Net-(D39-A)
Other:
- board outline added: 321.8 x 269.5 mm
- board text added: "Z1 5V"

Commit message: made cleanup changes, put notes in doc
Parts:
- added D2: WS2812B, LED_SMD:LED_WS2812B_PLCC4_5.0x5.0mm_P3.2mm, F.Cu at (310.6, -40.7)
- added D21: WS2812B, LED_SMD:LED_WS2812B_PLCC4_5.0x5.0mm_P3.2mm, F.Cu at (318.7, -27.4)
- added D22: WS2812B, LED_SMD:LED_WS2812B_PLCC4_5.0x5.0mm_P3.2mm, F.Cu at (318.7, -20.8)
- added D24: WS2812B, LED_SMD:LED_WS2812B_PLCC4_5.0x5.0mm_P3.2mm, F.Cu at (318.7, -14.2)
- added D25: WS2812B, LED_SMD:LED_WS2812B_PLCC4_5.0x5.0mm_P3.2mm, F.Cu at (326.8, -40.7)
- added D26: WS2812B, LED_SMD:LED_WS2812B_PLCC4_5.0x5.0mm_P3.2mm, F.Cu at (326.8, -34.1)
- added D27: WS2812B, LED_SMD:LED_WS2812B_PLCC4_5.0x5.0mm_P3.2mm, F.Cu at (326.8, -27.4)
- added D3: WS2812B, LED_SMD:LED_WS2812B_PLCC4_5.0x5.0mm_P3.2mm, F.Cu at (310.6, -34.1)
- added D4: WS2812B, LED_SMD:LED_WS2812B_PLCC4_5.0x5.0mm_P3.2mm, F.Cu at (310.6, -27.4)
- added D5: WS2812B, LED_SMD:LED_WS2812B_PLCC4_5.0x5.0mm_P3.2mm, F.Cu at (310.6, -20.8)
- added D6: WS2812B, LED_SMD:LED_WS2812B_PLCC4_5.0x5.0mm_P3.2mm, F.Cu at (310.6, -14.2)
- added D7: WS2812B, LED_SMD:LED_WS2812B_PLCC4_5.0x5.0mm_P3.2mm, F.Cu at (318.7, -40.7)
- added D8: WS2812B, LED_SMD:LED_WS2812B_PLCC4_5.0x5.0mm_P3.2mm, F.Cu at (318.7, -34.1)
Connections:
- J5 pad 12: unconnected-(J5-GPIO18/SPI1_~{CE0}/PCM_CLK/PWM0-Pad12) -> Net-(J16-Pin_2)
- J5 pad 38: unconnected-(J5-GPIO20/SPI1_MOSI/PCM_DIN/PWM1-Pad38) -> Net-(J17-Pin_2)
- LS1 pad 1: unconnected-(LS1-Pad1) -> Net-(U7-PA5)
- LS1 pad 2: unconnected-(LS1-Pad2) -> GND
- U20 pad 15: unconnected-(U20-SENSE_B-Pad15) -> GND
- U3 pad 21: unconnected-(U3-PA5-Pad21) -> Net-(U3-PA5)
- U3 pad 36: unconnected-(U3-PB15-Pad36) -> Net-(D8-DIN)
- U7 pad 21: unconnected-(U7-PA5-Pad21) -> Net-(U7-PA5)
- U7 pad 36: unconnected-(U7-PB15-Pad36) -> Net-(D2-DIN)

Commit message: Small updates.
Parts:
- removed the D2 at (44.0, -59.6)
- removed the D21 at (52.2, -46.4)
- removed the D22 at (52.2, -39.8)
- removed the D24 at (52.2, -33.2)
- removed the D25 at (60.3, -59.6)
- removed the D26 at (60.3, -53.0)
- removed the D27 at (60.3, -46.4)
- removed the D3 at (44.0, -53.0)
- removed the D4 at (44.0, -46.4)
- removed the D5 at (44.0, -39.8)
- removed the D6 at (44.0, -33.2)
- removed the D7 at (52.2, -59.6)
- removed the D8 at (52.2, -53.0)
- removed LS2: BUZZER, PS1240P02BT:XDCR_PS1240P02BT
- removed R37, R44, R50, R56, R62, R77: 53, Resistor_SMD:R_0603_1608Metric
- removed REF**: MODULE_RASPBERRY_PI_4B_4GB, RASPBERRY_PI_4B_4GB:MODULE_RASPBERRY_PI_4B_4GB
- moved R97 424.1 mm to (103.3, -262.2), turned to 90 degrees
- moved R98 422.5 mm to (111.8, -262.2), turned to 90 degrees
- moved D54 418.5 mm to (109.8, -262.2), turned to 90 degrees
- moved D53 418.0 mm to (105.3, -262.2), turned to 90 degrees
- moved R95 388.3 mm to (245.8, -262.2), turned to 90 degrees
- moved D51 387.3 mm to (247.8, -262.2), turned to 90 degrees
- moved R96 377.8 mm to (254.3, -262.2), turned to 90 degrees
- moved D52 376.9 mm to (252.3, -262.2), turned to 90 degrees
- moved D46 235.7 mm to (372.5, -91.0), turned to 90 degrees
- moved D45 231.5 mm to (368.0, -91.0), turned to 90 degrees
- moved R90 231.4 mm to (374.5, -91.0), turned to 90 degrees
- moved R89 226.0 mm to (366.0, -91.0), turned to 90 degrees
- moved R91 209.2 mm to (85.7, 75.3), turned to 90 degrees
- moved R92 201.3 mm to (94.2, 75.3), turned to 90 degrees
- moved D47 195.4 mm to (87.7, 75.3), turned to 90 degrees
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Connections:
- C29 pad 1: Net-(C29-Pad1) -> Net-(D40-A)
- C37 pad 1: Net-(C37-Pad1) -> Net-(D39-A)
- C44 pad 1: Net-(C44-Pad1) -> Net-(D41-A)
- C51 pad 1: Net-(C51-Pad1) -> Net-(D36-A)
- C58 pad 1: Net-(C58-Pad1) -> Net-(D38-A)
- C82 pad 1: Net-(C82-Pad1) -> Net-(D37-A)
- R22 pad 2: Net-(C29-Pad1) -> Net-(D40-A)
- R42 pad 2: Net-(C37-Pad1) -> Net-(D39-A)
- R48 pad 2: Net-(C44-Pad1) -> Net-(D41-A)
- R54 pad 2: Net-(C51-Pad1) -> Net-(D36-A)
- R60 pad 2: Net-(C58-Pad1) -> Net-(D38-A)
- R75 pad 2: Net-(C82-Pad1) -> Net-(D37-A)
Routing:
- net +3.3V_Z1: track 47.5 -> 11.3 mm
- net +3.3V_Z2: track 47.4 -> 11.3 mm
- net +3.3V_Z3: track 47.4 -> 11.3 mm
- net /Z1_SCLK: track 29.3 -> 5.33 mm
- net /Z3_SCLK: track 29.3 -> 5.32 mm
- net /Z2_SCLK: track 29.3 -> 5.33 mm
- net /Z1_MOSI: track 25.7 -> 4.63 mm
- net /Z3_MOSI: track 25.7 -> 4.63 mm
- net /Z2_MOSI: track 25.7 -> 4.63 mm
- net /Z1_MISO: track 24.1 -> 4.80 mm
- net /Z2_MISO: track 24.1 -> 4.80 mm
- net /Z3_MISO: track 24.1 -> 4.80 mm
- net GND: track 161.3 -> 142.9 mm, vias 116 -> 96
- net Net-(D43-A): track 27.9 -> 12.2 mm, vias 2 -> 0
- net /Z3_INT_CAN_B: track 15.4 -> 2.58 mm
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- added copper zone on F.Cu, net Net-(IC1-SW)
- added copper zone on F.Cu, net Net-(IC1-VIN)
- added copper zone on F.Cu, net Net-(IC2-SW)
- added copper zone on F.Cu, net Net-(IC2-VIN)
- added copper zone on F.Cu, net Net-(IC3-SW)
- added copper zone on F.Cu, net Net-(IC3-VIN)
- added copper zone on F.Cu, net Net-(IC4-SW)
- added copper zone on F.Cu, net Net-(IC4-VIN)
- added copper zone on F.Cu, net Net-(IC5-SW)
- added copper zone on F.Cu, net Net-(IC5-VIN)
- added copper zone on F.Cu, net Net-(IC6-SW)
- added copper zone on F.Cu, net Net-(IC6-VIN)
Other:
- board size 321.8 x 269.5 mm -> 337.8 x 269.5 mm

Commit message: Zone 2 complete
Parts:
- removed JP30: STM_POWER, Connector_PinHeader_2.54mm:PinHeader_1x02_P2.54mm_Vertical
- removed R67, R68, R8, R9: 0, Resistor_SMD:R_0603_1608Metric
- removed TP32: Z3_ERR, TestPoint:TestPoint_Keystone_5015_Micro_Mini
- removed TP33: Z1_CANL_A, TestPoint:TestPoint_Keystone_5015_Micro_Mini
- removed TP34: Z1_CANH_A, TestPoint:TestPoint_Keystone_5015_Micro_Mini
- removed TP35: Z1_CANH_B, TestPoint:TestPoint_Keystone_5015_Micro_Mini
- removed TP36: Z1_CANL_B, TestPoint:TestPoint_Keystone_5015_Micro_Mini
- removed TP37: Z2_CANH_B, TestPoint:TestPoint_Keystone_5015_Micro_Mini
- removed TP38: Z2_CANL_B, TestPoint:TestPoint_Keystone_5015_Micro_Mini
- removed TP39: Z2_CANH_A, TestPoint:TestPoint_Keystone_5015_Micro_Mini
- removed TP40: Z2_CANL_A, TestPoint:TestPoint_Keystone_5015_Micro_Mini
- removed TP41: Z3_CANH_B, TestPoint:TestPoint_Keystone_5015_Micro_Mini
- removed TP42: Z3_CANL_B, TestPoint:TestPoint_Keystone_5015_Micro_Mini
- removed TP43: Z3_CANH_A, TestPoint:TestPoint_Keystone_5015_Micro_Mini
- removed TP44: Z3_CANL_A, TestPoint:TestPoint_Keystone_5015_Micro_Mini
- added C100: 0.1uF, Capacitor_SMD:C_0603_1608Metric, F.Cu at (193.1, -120.8)
- added C88: 0.1uF, Capacitor_SMD:C_0603_1608Metric, F.Cu at (163.0, -386.6)
- added C89: 0.1uF, Capacitor_SMD:C_0603_1608Metric, F.Cu at (163.0, -384.0)
- added C90: 0.1uF, Capacitor_SMD:C_0603_1608Metric, F.Cu at (266.9, -401.5)
- added C91: 0.1uF, Capacitor_SMD:C_0603_1608Metric, F.Cu at (266.9, -399.0)
- added C92: 0.1uF, Capacitor_SMD:C_0603_1608Metric, F.Cu at (176.4, -90.8)
- added C93: 0.1uF, Capacitor_SMD:C_0603_1608Metric, F.Cu at (177.4, -74.0)
- added C94: 0.1uF, Capacitor_SMD:C_0603_1608Metric, F.Cu at (185.2, -75.8)
- added C95: 0.1uF, Capacitor_SMD:C_0603_1608Metric, F.Cu at (187.0, -87.5)
- added C96: 0.1uF, Capacitor_SMD:C_0603_1608Metric, F.Cu at (170.4, -80.5)
- added C97: 1uF, Capacitor_SMD:C_0603_1608Metric, F.Cu at (170.4, -78.8)
- added C98: 0.1uF, Capacitor_SMD:C_0603_1608Metric, F.Cu at (107.7, -289.8)
- added C99: 1uF, Capacitor_SMD:C_0603_1608Metric, F.Cu at (274.9, -409.1)
- added J16: Conn_01x03_Pin, Connector_PinHeader_2.54mm:PinHeader_1x03_P2.54mm_Vertical, F.Cu at (388.6, -129.6)
- added J17: Conn_01x03_Pin, Connector_PinHeader_2.54mm:PinHeader_1x03_P2.54mm_Vertical, F.Cu at (393.2, -129.6)
- added JP2: 3.3 Souce, Jumper:SolderJumper-3_P1.3mm_Bridged12_RoundedPad1.0x1.5mm_NumberLabels, F.Cu at (389.1, -120.4)
- added JP34: STM_POWER, Connector_PinHeader_2.54mm:PinHeader_1x02_P2.54mm_Vertical, F.Cu at (279.5, -389.5)
- added LS2: BUZZER, PS1240P02BT:XDCR_PS1240P02BT, F.Cu at (234.4, -336.6)
- added R44: 10k, Resistor_SMD:R_0603_1608Metric, F.Cu at (163.0, -381.5)
- added R50: 10k, Resistor_SMD:R_0603_1608Metric, F.Cu at (163.0, -379.0)
- added R56: 10k, Resistor_SMD:R_0603_1608Metric, F.Cu at (163.0, -376.5)
- added R62: 10k, Resistor_SMD:R_0603_1608Metric, F.Cu at (163.0, -374.0)
- added R77: 120, Resistor_SMD:R_0603_1608Metric, F.Cu at (196.1, -120.8)
- added TP56: GND, TestPoint:TestPoint_Keystone_5015_Micro_Mini, F.Cu at (295.7, -300.3)
- added TP57: GND, TestPoint:TestPoint_Keystone_5015_Micro_Mini, F.Cu at (419.2, -200.1)
- added TP58: GND, TestPoint:TestPoint_Keystone_5015_Micro_Mini, F.Cu at (194.1, -52.4)
- added TP59: DIR_A, TestPoint:TestPoint_Keystone_5015_Micro_Mini, F.Cu at (106.5, -485.6)
- added TP60: MOTOR_LEFT_PWM, TestPoint:TestPoint_Keystone_5015_Micro_Mini, F.Cu at (106.5, -481.8)
- added TP61: ERR, TestPoint:TestPoint_Keystone_5015_Micro_Mini, F.Cu at (106.5, -478.1)
- added TP62: SERVO_PWM, TestPoint:TestPoint_Keystone_5015_Micro_Mini, F.Cu at (186.4, -112.3)
- added TP63: RR, TestPoint:TestPoint_Keystone_5015_Micro_Mini, F.Cu at (217.7, -347.8)
- added TP64: RL, TestPoint:TestPoint_Keystone_5015_Micro_Mini, F.Cu at (217.7, -344.1)
- added TP65: DEG_B, TestPoint:TestPoint_Keystone_5015_Micro_Mini, F.Cu at (217.7, -340.3)
- added TP66: DEG_A, TestPoint:TestPoint_Keystone_5015_Micro_Mini, F.Cu at (217.7, -336.6)
- added TP67: DEG_A, TestPoint:TestPoint_Keystone_5015_Micro_Mini, F.Cu at (196.2, -66.3)
- added TP68: DEG_B, TestPoint:TestPoint_Keystone_5015_Micro_Mini, F.Cu at (195.9, -59.8)
- added TP69: FL, TestPoint:TestPoint_Keystone_5015_Micro_Mini, F.Cu at (126.2, -92.3)
- added TP70: FR, TestPoint:TestPoint_Keystone_5015_Micro_Mini, F.Cu at (230.7, -92.3)
- added TP71: ERR, TestPoint:TestPoint_Keystone_5015_Micro_Mini, F.Cu at (196.4, -73.0)
- added TP72: DEG_A, TestPoint:TestPoint_Keystone_5015_Micro_Mini, F.Cu at (373.7, -162.8)
- added TP73: DEG_B, TestPoint:TestPoint_Keystone_5015_Micro_Mini, F.Cu at (373.7, -159.1)
- added TP74: ERR, TestPoint:TestPoint_Keystone_5015_Micro_Mini, F.Cu at (356.9, -148.6)
- added TP75: CUR_POST, TestPoint:TestPoint_Keystone_5015_Micro_Mini, F.Cu at (188.3, -120.8)
- added TP76: GND, TestPoint:TestPoint_Keystone_5015_Micro_Mini, F.Cu at (179.0, -52.2)
- added TP77: GND, TestPoint:TestPoint_Keystone_5015_Micro_Mini, F.Cu at (164.2, -51.8)
- added TP78: GND, TestPoint:TestPoint_Keystone_5015_Micro_Mini, F.Cu at (216.8, -88.0)
- added TP79: GND, TestPoint:TestPoint_Keystone_5015_Micro_Mini, F.Cu at (141.2, -121.2)
- C62: value 1uF -> 0.1uF
- C74: value 0.1uF -> 1uF
- D10, D15, D20: value DEGRADED -> DEGRADED_B
- D14, D19, D9: value DEGRADED -> DEGRADED_A
- FB1, FB2: footprint Inductor_SMD:L_0201_0603Metric -> Inductor_SMD:L_0603_1608Metric
- JP1, JP11, JP19, JP9: value ~ -> TERM
- R75: value 91K -> 510K
- R76: value 10K -> 47K
- TP101: renamed from Z2_CAN_TX_A1; value CMD_TX -> Z2_CAN_TX_A
- TP15: value MOTOR_PWM_OUT -> MOTOR_RIGHT_PWM
- TP47: value SERVO_CURRENT -> CURR_PRE
- TP48: value Z3_5_EN -> Z2_5_EN
- TP8: value Z2_CAN_RX_B -> Z2_CAN_TX_B
- moved D21 269.5 mm to (272.9, -293.1)
- moved D22 269.5 mm to (272.9, -286.5)
- moved D24 269.5 mm to (272.9, -279.8)
- moved D25 269.5 mm to (281.0, -306.3)
- moved D26 269.5 mm to (281.0, -299.7)
- moved D27 269.5 mm to (281.0, -293.1)
- moved D8 269.5 mm to (272.9, -299.7)
- moved JP33 247.9 mm to (175.9, -120.0), turned to 90 degrees
- moved TP49 245.5 mm to (171.4, -120.3), turned to 180 degrees
- moved R71 245.5 mm to (192.8, -116.0), turned to 0 degrees
- moved TP53 242.0 mm to (132.8, -100.4), turned to 180 degrees
- moved TP52 239.9 mm to (161.8, -120.0), turned to 180 degrees
- moved D37 239.1 mm to (179.3, -114.0), turned to 90 degrees
- moved JP11 237.8 mm to (127.2, -99.5), turned to 180 degrees
- moved R10 237.7 mm to (131.8, -97.4), turned to 90 degrees
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Connections:
- net Net-(JP31-A) renamed /STM_POWER_Z2
- C62 pad 1: Net-(JP30-A) -> /STM_POWER_Z3
- C65 pad 2: Net-(C65-Pad2) -> Net-(U3-PC14)
- C66 pad 1: Net-(C66-Pad1) -> Net-(U3-PC15)
- C68 pad 2: Net-(C68-Pad2) -> Net-(U7-PC14)
- C69 pad 1: Net-(C69-Pad1) -> Net-(U7-PC15)
- C74 pad 1: /MOTOR_CURRENT_LEFT -> /STM_POWER_Z3
- C77 pad 1: /MOTOR_CURRENT_RIGHT -> /STM_POWER_Z3
- D2 pad 1: +5V_Z1 -> +7V_Z2
- D3 pad 1: +5V_Z1 -> +7V_Z2
- D4 pad 1: +5V_Z1 -> +7V_Z2
- D5 pad 1: +5V_Z1 -> +7V_Z2
- D6 pad 1: +5V_Z1 -> +7V_Z2
- D7 pad 1: +5V_Z1 -> +7V_Z2
- J2 pad 6: /Z3_SCLK -> /Z3_SWO
- J3 pad 6: /Z2_SCLK -> /Z2_SWO
- J5 pad 27: unconnected-(J5-ID_SD_I2C0/GPIO00-Pad27) -> /Z1_TEST_BUTTON
- LS1 pad 1: Net-(U7-PA5) -> Net-(U7-PA15)
- TP47 pad 1: /SERVO_CURRENT -> Net-(R77-Pad1)
- U3 pad 1: Net-(JP30-A) -> /STM_POWER_Z3
- U3 pad 19: Net-(JP30-A) -> /STM_POWER_Z3
- U3 pad 21: Net-(U3-PA5) -> /Z3_SCLK
- U3 pad 32: Net-(JP30-A) -> /STM_POWER_Z3
- U3 pad 48: Net-(JP30-A) -> /STM_POWER_Z3
- U3 pad 55: /Z3_SCLK -> /Z3_SWO
- U3 pad 64: Net-(JP30-A) -> /STM_POWER_Z3
- U5 pad 1: /SERVO_CURRENT -> Net-(R77-Pad1)
- U7 pad 21: Net-(U7-PA5) -> /Z2_SCLK
- U7 pad 50: unconnected-(U7-PA15-Pad50) -> Net-(U7-PA15)
- U7 pad 55: /Z2_SCLK -> /Z2_SWO
- Y7 pad 1: Net-(C65-Pad2) -> Net-(U3-PC14)
- Y7 pad 4: Net-(C66-Pad1) -> Net-(U3-PC15)
- Y8 pad 1: Net-(C68-Pad2) -> Net-(U7-PC14)
- Y8 pad 4: Net-(C69-Pad1) -> Net-(U7-PC15)
Routing:
- net +7V_Z2: track 0.00 -> 215.5 mm, vias 0 -> 2
- net +3.3V_Z2: track 11.3 -> 171.0 mm, vias 0 -> 5
- net /SERVO_CURRENT: track 0.00 -> 141.0 mm, vias 0 -> 2
- net Net-(D2-DIN): track 0.00 -> 117.0 mm, vias 0 -> 2
- net GND: track 142.9 -> 242.3 mm, vias 96 -> 129
- net +12V: track 0.00 -> 97.6 mm, vias 0 -> 3
- net /Z2_SCLK: track 5.33 -> 90.9 mm, vias 0 -> 3
- net /SERVO_PWM: track 0.00 -> 85.3 mm, vias 0 -> 2
- net /Z2_MOSI: track 4.63 -> 78.8 mm
- net (no net): track 0.00 -> 74.0 mm
- net /Z2_MISO: track 4.80 -> 77.9 mm, vias 0 -> 2
- net /FR_BLINK: track 0.00 -> 71.4 mm
- net /Z2_NRST: track 0.00 -> 68.9 mm, vias 0 -> 1
- net /FL_BLINK: track 0.00 -> 67.6 mm, vias 0 -> 2
- net /STM_POWER_Z2: track 0.00 -> 65.1 mm, vias 0 -> 4
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Other:
- board size 337.8 x 269.5 mm -> 121.5 x 269.9 mm
- board text added: "HIGH"
- board text added: "LOW"

Commit message: Most of Z3 routed.
Parts:
- moved D28 251.5 mm to (136.0, -235.4), turned to 90 degrees
- moved D29 240.5 mm to (156.0, -235.6), turned to 90 degrees
- moved D32 237.6 mm to (136.0, -227.9), turned to 90 degrees
- moved D30 229.1 mm to (201.3, -234.9), turned to 90 degrees
- moved D33 226.3 mm to (156.1, -228.1), turned to 90 degrees
- moved D31 223.5 mm to (221.3, -234.7), turned to 90 degrees
- moved D34 214.4 mm to (201.3, -227.4), turned to 90 degrees
- moved D35 208.8 mm to (221.3, -227.2), turned to 90 degrees
- moved J7 188.1 mm to (141.0, -230.4), turned to 0 degrees
- moved J8 177.4 mm to (206.3, -229.7), turned to 0 degrees
- moved U20 176.6 mm to (169.8, -231.5)
- moved C26 176.2 mm to (194.5, -254.2), turned to 90 degrees
- moved TP12 176.0 mm to (128.4, -252.0), turned to 180 degrees
- moved R38 175.2 mm to (132.8, -252.1), turned to 90 degrees
- moved C34 174.4 mm to (137.9, -252.4), turned to -90 degrees
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Connections:
- net Net-(D28-K) renamed /MOTOR_PWR+_R
- net Net-(D29-K) renamed /MOTOR_PWR-_R
- net Net-(D30-K) renamed /MOTOR_PWR-_L
- net Net-(D31-K) renamed /MOTOR_PWR+_L
- net Net-(J7-Pin_1) renamed /MOTOR_PWR+C_R
- net Net-(J8-Pin_6) renamed /MOTOR_PWR+C_L
- JP19 pad 1: /CANH_B -> /CANL_B
- R21 pad 1: Net-(JP19-B) -> /CANH_B
- R21 pad 2: /CANL_B -> Net-(JP19-B)
- U3 pad 11: /MOTOR_CURRENT_LEFT -> /MOTOR_CURRENT_RIGHT
- U3 pad 24: /MOTOR_CURRENT_RIGHT -> /MOTOR_CURRENT_LEFT
Routing:
- net +12V: track 97.6 -> 322.8 mm, vias 3 -> 9
- net +5V_Z3: track 0.00 -> 165.6 mm, vias 0 -> 6
- net /ENC_LEFT_B: track 0.00 -> 121.1 mm, vias 0 -> 4
- net /Z3_SCLK: track 5.32 -> 124.1 mm, vias 0 -> 4
- net /Z3_MOSI: track 4.63 -> 106.9 mm
- net /Z3_MISO: track 4.80 -> 104.8 mm, vias 0 -> 2
- net +5V_Z1: track 0.00 -> 94.2 mm
- net /Z3_TEST_BUTTON: track 0.00 -> 88.5 mm, vias 0 -> 2
- net /ENC_LEFT_A: track 0.00 -> 78.0 mm, vias 0 -> 2
- net /MOTOR_RIGHT_PWM: track 0.00 -> 75.3 mm, vias 0 -> 6
- net /Z3_INT_CAN_B: track 2.58 -> 76.1 mm, vias 0 -> 2
- net /MOTOR_CURRENT_LEFT: track 0.00 -> 72.0 mm, vias 0 -> 2
- net /ENC_RIGHT_A: track 0.00 -> 70.1 mm, vias 0 -> 2
- net /ENC_RIGHT_B: track 0.00 -> 69.3 mm, vias 0 -> 4
- net /MOTOR_CURRENT_RIGHT: track 0.00 -> 67.1 mm, vias 0 -> 2
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