File: lab4/Schematic/Schematic.kicad_pcb (KiCad board)
At the start: 2 copper layers, 121.5 x 269.9 mm, 399 parts, among them IC1 TPS564252DRLR, IC2 TPS564252DRLR, IC3 TPS564252DRLR, IC4 TPS564252DRLR, IC5 TPS564252DRLR, IC6 TPS564252DRLR, J1 XT60-M, J10 CANA_Z1, J11 CANA_Z1, J12 CANA_Z1, J13 CANA_Z1, J14 CANA_Z1, J15 CANA_Z1, J16 Conn_01x03_Pin, J17 Conn_01x03_Pin, J2 Z2_SWD, J3 Z2_SWD, J4 Z3_USART, J5 Raspberry_Pi_4, J6 Z3_USART, J7 MOTOR_RIGHT, J8 MOTOR_LEFT, J9 SERVO, Q2 IRF4905, U1 MCP2515-xST, U10 SN65HVD230, U11 MCP2515-xST, U12 SN65HVD230, U13 MCP2515-xST, U14 SN65HVD230, U15 MCP2515-xST, U16 SN65HVD230, U17 MCP2515-xST, U18 SN65HVD230, U2 ACS712xLCTR-05B, U20 L298N, U3 STM32F401RETx, U4 ACS712xLCTR-05B, U5 INA181, U7 STM32F401RETx, U8 SN65HVD230, U9 MCP2515-xST, Y1 CX3225SB16000H0FLJCC, Y2 CX3225SB16000H0FLJCC, Y3 CX3225SB16000H0FLJCC, Y4 CX3225SB16000H0FLJCC, Y5 CX3225SB16000H0FLJCC, Y6 CX3225SB16000H0FLJCC, Y7 ABS25-32.768KHZ-6-T, Y8 ABS25-32.768KHZ-6-T

Commit message: Initial Board layout complete and DRC passes
Parts:
- removed TP31: Z3_ERR, TestPoint:TestPoint_Keystone_5015_Micro_Mini
- added J18: Barrel_Jack, Connector_BarrelJack:BarrelJack_Horizontal, F.Cu at (207.0, -141.2)
- added JP3: PIXEL POWER, Jumper:SolderJumper-2_P1.3mm_Bridged_RoundedPad1.0x1.5mm, F.Cu at (222.7, -79.0)
- added JP4: SolderJumper_2_Bridged, Jumper:SolderJumper-2_P1.3mm_Bridged_RoundedPad1.0x1.5mm, F.Cu at (236.3, -297.8)
- added TP80: GND, TestPoint:TestPoint_Keystone_5015_Micro_Mini, F.Cu at (134.0, -295.8)
- added TP81: GND, TestPoint:TestPoint_Keystone_5015_Micro_Mini, F.Cu at (228.0, -240.8)
- added TP82: GND, TestPoint:TestPoint_Keystone_5015_Micro_Mini, F.Cu at (125.0, -242.0)
- added TP83: GND, TestPoint:TestPoint_Keystone_5015_Micro_Mini, F.Cu at (153.0, -265.8)
- added TP84: GND, TestPoint:TestPoint_Keystone_5015_Micro_Mini, F.Cu at (124.8, -203.8)
- added TP85: GND, TestPoint:TestPoint_Keystone_5015_Micro_Mini, F.Cu at (226.2, -197.5)
- added TP86: GND, TestPoint:TestPoint_Keystone_5015_Micro_Mini, F.Cu at (166.2, -139.5)
- TP16: value Z3_CAN_TX_A -> CAN_TX_A
- TP18: value Z3_CAN_RX_A -> CAN_RX_A
- TP19: value Z3_CAN_RX_B -> CAN_RX_B
- moved R47 310.8 mm to (155.8, -197.2), turned to 90 degrees
- moved TP50 309.9 mm to (156.8, -200.2), turned to 180 degrees
- moved C44 309.0 mm to (155.8, -191.2), turned to -90 degrees
- moved R49 306.0 mm to (156.9, -188.3), turned to 180 degrees
- moved R48 305.1 mm to (157.8, -191.2), turned to 90 degrees
- moved TP21 301.3 mm to (158.8, -182.5), turned to 180 degrees
- moved C46 299.4 mm to (161.6, -197.6), turned to 180 degrees
- moved C43 299.0 mm to (160.2, -185.7), turned to 90 degrees
- moved C45 298.7 mm to (161.6, -195.4), turned to 180 degrees
- moved C47 298.0 mm to (161.6, -193.5), turned to 180 degrees
- moved IC3 297.1 mm to (161.6, -190.0), turned to 180 degrees
- moved R46 293.1 mm to (163.2, -185.6), turned to 90 degrees
- moved R45 292.5 mm to (163.2, -182.6), turned to 90 degrees
- moved TP22 291.2 mm to (166.4, -200.5), turned to 180 degrees
- moved C42 286.5 mm to (166.2, -183.0), turned to -90 degrees
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Connections:
- D2 pad 1: +7V_Z2 -> Net-(D2-VDD)
- D21 pad 1: +5V_Z1 -> Net-(D21-VDD)
- D22 pad 1: +5V_Z1 -> Net-(D21-VDD)
- D24 pad 1: +5V_Z1 -> Net-(D21-VDD)
- D25 pad 1: +5V_Z1 -> Net-(D21-VDD)
- D26 pad 1: +5V_Z1 -> Net-(D21-VDD)
- D27 pad 1: +5V_Z1 -> Net-(D21-VDD)
- D3 pad 1: +7V_Z2 -> Net-(D2-VDD)
- D4 pad 1: +7V_Z2 -> Net-(D2-VDD)
- D5 pad 1: +7V_Z2 -> Net-(D2-VDD)
- D6 pad 1: +7V_Z2 -> Net-(D2-VDD)
- D7 pad 1: +7V_Z2 -> Net-(D2-VDD)
- D8 pad 1: +5V_Z1 -> Net-(D21-VDD)
- J1 pad 1: (no net) -> GND
- J1 pad 2: (no net) -> Net-(J1-POS)
Routing:
- net +3.3V_Z3: track 33.6 -> 206.5 mm
- net /CANH_B: track 36.0 -> 200.6 mm
- net /CANL_B: track 40.7 -> 204.1 mm
- net /CANH_A: track 45.2 -> 205.5 mm
- net /CANL_A: track 52.0 -> 205.7 mm, vias 0 -> 1
- net +12V: track 322.8 -> 471.8 mm, vias 9 -> 11
- net +3.3V_Z1: track 11.3 -> 152.3 mm, vias 0 -> 2
- net +7V_Z2: track 215.5 -> 99.2 mm
- net Net-(D2-VDD): track 0.00 -> 115.7 mm
- net /Z1_MISO: track 4.80 -> 118.9 mm, vias 0 -> 1
- net Net-(D21-VDD): track 0.00 -> 111.9 mm
- net /Z1_SCLK: track 5.32 -> 113.2 mm
- net /Z1_MOSI: track 4.63 -> 108.2 mm, vias 0 -> 2
- net /PI_3.3V: track 0.00 -> 96.8 mm, vias 0 -> 5
- net Net-(D8-DIN): track 0.00 -> 94.3 mm, vias 0 -> 4
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Other:
- outline, holes or cut-outs redrawn
