File: lab4/Schematic/Schematic.kicad_pcb (KiCad board)
At the start: 2 copper layers, 121.5 x 269.9 mm, 408 parts, among them IC1 TPS564252DRLR, IC2 TPS564252DRLR, IC3 TPS564252DRLR, IC4 TPS564252DRLR, IC5 TPS564252DRLR, IC6 TPS564252DRLR, J1 XT60-M, J10 CANA_Z1, J11 CANA_Z1, J12 CANA_Z1, J13 CANA_Z1, J14 CANA_Z1, J15 CANA_Z1, J16 Conn_01x03_Pin, J17 Conn_01x03_Pin, J18 Barrel_Jack, J2 Z2_SWD, J3 Z2_SWD, J4 Z3_USART, J5 Raspberry_Pi_4, J6 Z3_USART, J7 MOTOR_RIGHT, J8 MOTOR_LEFT, J9 SERVO, Q2 IRF4905, U1 MCP2515-xST, U10 SN65HVD230, U11 MCP2515-xST, U12 SN65HVD230, U13 MCP2515-xST, U14 SN65HVD230, U15 MCP2515-xST, U16 SN65HVD230, U17 MCP2515-xST, U18 SN65HVD230, U2 ACS712xLCTR-05B, U20 L298N, U3 STM32F401RETx, U4 ACS712xLCTR-05B, U5 INA181, U7 STM32F401RETx, U8 SN65HVD230, U9 MCP2515-xST, Y1 CX3225SB16000H0FLJCC, Y2 CX3225SB16000H0FLJCC, Y3 CX3225SB16000H0FLJCC, Y4 CX3225SB16000H0FLJCC, Y5 CX3225SB16000H0FLJCC, Y6 CX3225SB16000H0FLJCC, Y7 ABS25-32.768KHZ-6-T, Y8 ABS25-32.768KHZ-6-T

Commit message: Logic level and v-reg for leds. Motor Driver heatsink. Fixed pth vs sm footprints. Misc.
Parts:
- added C101: 4.7uF, Capacitor_SMD:C_0805_2012Metric, F.Cu at (218.1, -89.1)
- added C102: 4.7uF, Capacitor_SMD:C_0805_2012Metric, F.Cu at (220.8, -82.8)
- added HS1: 6396BG, 449proj:HSINK_6396BG, F.Cu at (178.5, -253.9)
- added Q1: 2N7002, Package_TO_SOT_SMD:SOT-23, F.Cu at (157.1, -58.5)
- added Q3: 2N7002, Package_TO_SOT_SMD:SOT-23, F.Cu at (217.5, -311.5)
- added R100: 4K7, Resistor_SMD:R_0603_1608Metric, F.Cu at (154.2, -57.6)
- added R101: 4K7, Resistor_SMD:R_0603_1608Metric, F.Cu at (214.5, -311.5)
- added R102: 4K7, Resistor_SMD:R_0603_1608Metric, F.Cu at (218.0, -314.0)
- added R37: 10k, Resistor_SMD:R_0603_1608Metric, F.Cu at (221.7, -81.1)
- added R67: 47K, Resistor_SMD:R_0603_1608Metric, F.Cu at (219.5, -80.4)
- added R68: 4K7, Resistor_SMD:R_0603_1608Metric, F.Cu at (218.0, -80.4)
- added R99: 4K7, Resistor_SMD:R_0603_1608Metric, F.Cu at (160.1, -58.5)
- added REF**: TestPoint_Pad_D1.0mm, TestPoint:TestPoint_Pad_D1.0mm, F.Cu at (191.2, -293.2)
- added REF**: TestPoint_Pad_D1.0mm, TestPoint:TestPoint_Pad_D1.0mm, F.Cu at (213.2, -288.5)
- added REF**: TestPoint_Pad_D1.0mm, TestPoint:TestPoint_Pad_D1.0mm, F.Cu at (149.1, -289.2)
- added REF**: TestPoint_Pad_D1.0mm, TestPoint:TestPoint_Pad_D1.0mm, F.Cu at (211.2, -288.5)
- added REF**: TestPoint_Pad_D1.0mm, TestPoint:TestPoint_Pad_D1.0mm, F.Cu at (149.4, -285.6)
- added REF**: TestPoint_Pad_D1.0mm, TestPoint:TestPoint_Pad_D1.0mm, F.Cu at (178.0, -303.5)
- added REF**: TestPoint_Pad_D1.0mm, TestPoint:TestPoint_Pad_D1.0mm, F.Cu at (179.0, -300.8)
- added REF**: TestPoint_Pad_D1.0mm, TestPoint:TestPoint_Pad_D1.0mm, F.Cu at (189.2, -293.2)
- added REF**: TestPoint_Pad_D1.0mm, TestPoint:TestPoint_Pad_D1.0mm, F.Cu at (218.5, -288.8)
- added REF**: TestPoint_Pad_D1.0mm, TestPoint:TestPoint_Pad_D1.0mm, F.Cu at (148.2, -287.2)
- added REF**: TestPoint_Pad_D1.0mm, TestPoint:TestPoint_Pad_D1.0mm, F.Cu at (151.1, -289.6)
- added REF**: TestPoint_Pad_D1.0mm, TestPoint:TestPoint_Pad_D1.0mm, F.Cu at (150.2, -287.5)
- added REF**: TestPoint_Pad_D1.0mm, TestPoint:TestPoint_Pad_D1.0mm, F.Cu at (215.4, -288.6)
- added REF**: TestPoint_Pad_D1.0mm, TestPoint:TestPoint_Pad_D1.0mm, F.Cu at (147.2, -285.5)
- added REF**: TestPoint_Pad_D1.0mm, TestPoint:TestPoint_Pad_D1.0mm, F.Cu at (214.5, -286.5)
- added REF**: TestPoint_Pad_D1.0mm, TestPoint:TestPoint_Pad_D1.0mm, F.Cu at (216.5, -286.8)
- added REF**: TestPoint_Pad_D1.0mm, TestPoint:TestPoint_Pad_D1.0mm, F.Cu at (179.5, -305.5)
- added REF**: TestPoint_Pad_D1.0mm, TestPoint:TestPoint_Pad_D1.0mm, F.Cu at (181.2, -304.5)
- added REF**: TestPoint_Pad_D1.0mm, TestPoint:TestPoint_Pad_D1.0mm, F.Cu at (193.2, -293.2)
- added U6: AP7361EA-SPR-13, 449proj:AP7361EA_SO-8EP, F.Cu at (221.8, -87.3)
- C25, C26, C86: footprint Capacitor_THT:CP_Radial_D8.0mm_P3.80mm -> 449proj:CP_Elec_8x11.9_A768
- J7, J8: footprint Connector_JST:JST_PH_S6B-PH-K_1x06_P2.00mm_Horizontal -> Connector_JST:JST_PH_B6B-PH-SM4-TB_1x06-1MP_P2.00mm_Vertical
- moved TP60 42.0 mm to (202.0, -265.5)
- moved TP13 32.6 mm to (202.0, -260.5)
- moved C26 23.3 mm to (183.5, -233.7), turned to -90 degrees
- moved C25 23.2 mm to (173.5, -233.5), turned to -90 degrees
- moved R56 23.2 mm to (175.2, -278.5), turned to 180 degrees
- moved R50 22.7 mm to (178.9, -276.9), turned to 0 degrees
- moved R62 21.6 mm to (175.7, -276.9), turned to 180 degrees
- moved R44 21.5 mm to (178.1, -275.4), turned to 0 degrees
- moved C86 14.5 mm to (178.5, -261.5), turned to 90 degrees
- moved J2 12.7 mm to (182.0, -273.5)
- moved J4 11.7 mm to (192.0, -269.6)
- moved U20 11.5 mm to (169.6, -242.9)
- moved TP78 10.8 mm to (225.0, -95.0)
- moved JP3 10.8 mm to (212.0, -77.5), turned to 90 degrees
- moved TP15 8.96 mm to (174.5, -269.5)
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Connections:
- JP3 pad 2: +7V_Z2 -> Net-(JP3-B)
- U3 pad 2: /RR_BLINKER -> /RR_BLINK
- U3 pad 20: /MOTOR_LEFT_DIR -> /MOTOR_RIGHT_DIR
- U3 pad 22: /MOTOR_LEFT_PWM -> /MOTOR_RIGHT_PWM
- U3 pad 23: /MOTOR_RIGHT_PWM -> /MOTOR_LEFT_PWM
- U3 pad 25: /MOTOR_RIGHT_DIR -> /MOTOR_LEFT_DIR
- U3 pad 36: Net-(D8-DIN) -> Net-(Q3-S)
- U7 pad 36: Net-(D2-DIN) -> Net-(Q1-S)
Routing:
- net Net-(D2-DIN): track 117.0 -> 30.4 mm, vias 2 -> 0
- net Net-(Q1-S): track 0.00 -> 85.2 mm, vias 0 -> 2
- net Net-(Q3-S): track 0.00 -> 59.7 mm, vias 0 -> 4
- net Net-(D8-DIN): track 62.4 -> 6.32 mm, vias 4 -> 0
- net /RR_BLINK: track 2.66 -> 52.5 mm, vias 0 -> 2
- net +3.3V_Z2: track 171.0 -> 207.3 mm
- net +5V_Z3: track 239.4 -> 222.8 mm
- net +3.3V_Z3: track 207.0 -> 222.1 mm, vias 4 -> 6
- net /Z3_NRST: track 97.7 -> 83.7 mm
- net /Z3_SWO: track 45.5 -> 32.4 mm
- net Net-(D21-VDD): track 111.9 -> 124.9 mm
- net /Z3_TMS: track 35.0 -> 22.6 mm
- net /Z3_USART_TX: track 45.3 -> 33.8 mm
- net /MOTOR_LEFT_PWM: track 73.0 -> 61.6 mm, vias 3 -> 0
- net unconnected-(U3-PA10-Pad43): track 0.00 -> 10.8 mm
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- added copper zone on B.Cu, net +12V
- added copper zone on F.Cu, net +7V_Z2
- added copper zone on F.Cu, net Net-(JP3-B)

Commit message: Reworked ground at L298N
Parts:
- TP17: value Z3_CAN_TX_B -> CAN_TX_B
Routing:
- net +12V: track 465.1 -> 460.5 mm, vias 24 -> 16
- net /Z1_ERR: track 75.3 -> 75.8 mm
