File: lab4/Schematic/Schematic.kicad_sch (KiCad schematic)
At the start: 320 parts, among them IC1 TPS564252DRLR, IC2 TPS564252DRLR, IC3 TPS564252DRLR, IC4 TPS564252DRLR, IC5 TPS564252DRLR, IC6 TPS564252DRLR, J1 XT60-M, J10 CANA_Z1, J11 CANA_Z1, J12 CANA_Z1, J13 CANA_Z1, J14 CANA_Z1, J15 CANA_Z1, J2 Z2_SWD, J3 Z2_SWD, J4 Z3_USART, J5 Raspberry_Pi_4, J6 Z3_USART, J7 MOTOR_RIGHT, J8 MOTOR_LEFT, J9 SERVO, Q2 IRF4905, U1 MCP2515-xST, U10 SN65HVD230, U11 MCP2515-xST, U12 SN65HVD230, U13 MCP2515-xST, U14 SN65HVD230, U15 MCP2515-xST, U16 SN65HVD230, U17 MCP2515-xST, U18 SN65HVD230, U2 ACS712xLCTR-05B, U20 L298N, U3 STM32F401RETx, U4 ACS712xLCTR-05B, U5 INA181, U7 STM32F401RETx, U8 SN65HVD230, U9 MCP2515-xST, Y1 CX3225SB16000H0FLJCC, Y2 CX3225SB16000H0FLJCC, Y3 CX3225SB16000H0FLJCC, Y4 CX3225SB16000H0FLJCC, Y5 CX3225SB16000H0FLJCC, Y6 CX3225SB16000H0FLJCC, Y7 ABS25-32.768KHZ-6-T, Y8 ABS25-32.768KHZ-6-T

Commit message: Schematic 1.1 for small componet value issues
Parts:
- L1, L2, L3: value 2.2uH -> 3.3uH
- LS1, LS2: value PS1240P02BT -> BUZZER
- R75: value 330k -> 91K
- R76: value 30k -> 10K
Other:
- note removed: "Schematic is currently missing: - 6V power rail - Check the test points - Battery"
- title: CAN Lab Scheumatic  -> 18449 PCB LAB First Checkpoint
- moved on the sheet: LS2
Changed lines of the file:
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@@
 	(paper "D")
 	(title_block
-		(title "CAN Lab Scheumatic ")
-		(date "2026-10-22")
+		(title "18449 PCB LAB First Checkpoint")
+		(date "2026-10-25")
+		(rev "1.1")
 	)
 	(text "CAN controller schematic copied from: https://wiki.seeedstudio.com/xiao-can-bus-expansion"
@@
 		)
 	)
-	(text "Schematic is currently missing: \n- 6V power rail\n- Check the test points\n- Battery "
-		(exclude_from_sim no)
-		(at 778.256 494.03 0)
-		(effects
-			(font
-				(size 2.032 2.032)
-				(thickness 0.254)
-			)
-			(justify left)
-		)
-	)
 	(text "Notes: \n- AGND and GND are shared\n- This layout doens't have pin 31 or 47, but they should be \ntied to ground and that seems correct on the PCB. They are \npotentially suppsoed to have a 2.2 uF cap\n- The 8Mhz oscillator is not connected "
 		(exclude_from_sim no)
@@
 			)
 		)
-		(property "Value" "2.2uH"
+		(property "Value" "3.3uH"
 			(at 248.92 414.02 90)
 			(show_name no)
@@
 			)
 		)
-		(property "Value" "330k"
+		(property "Value" "91K"
 			(at 295.91 454.6599 0)
 			(show_name no)
@@
 			)
 		)
-		(property "Description" "Resistor, US symbol"
+		(property "Description" "RES 91K OHM 1% 1/10W 0603"
 			(at 293.37 453.39 0)
 			(hide yes)
@@
 			)
 		)
-		(property "Value" "2.2uH"
+		(property "Value" "3.3uH"
 			(at 71.12 415.29 90)
 			(show_name no)
@@
 			)
 		)
-		(property "Value" "2.2uH"
+		(property "Value" "3.3uH"
 			(at 433.07 416.56 90)
 			(show_name no)
@@
 			)
 		)
-		(property "Value" "30k"
+		(property "Value" "10K"
 			(at 295.656 467.36 0)
 			(show_name no)
@@
 			)
 		)
-		(property "Value" "PS1240P02BT"
+		(property "Value" "BUZZER"
 			(at 375.92 33.02 0)
 			(show_name no)
@@
 	(symbol
 		(lib_id "Device:PS1240P02BT")
-		(at 647.7 15.24 0)
+		(at 632.46 43.18 0)
 		(unit 1)
 		(body_style 1)
@@
 		(fields_autoplaced yes)
 		(property "Reference" "LS2"
-			(at 647.7 7.62 0)
+			(at 632.46 35.56 0)
 			(show_name no)
 			(do_not_autoplace no)
@@
 			)
 		)
-		(property "Value" "PS1240P02BT"
-			(at 647.7 10.16 0)
+		(property "Value" "BUZZER"
+			(at 632.46 38.1 0)
 			(show_name no)
 			(do_not_autoplace no)
@@
 		)
 		(property "Footprint" "PS1240P02BT:XDCR_PS1240P02BT"
-			(at 647.7 15.24 0)
+			(at 632.46 43.18 0)
 			(hide yes)
 			(show_name no)
@@
 		)
 		(property "Datasheet" ""
-			(at 647.7 15.24 0)
+			(at 632.46 43.18 0)
 			(hide yes)
 			(show_name no)
@@
 		)
 		(property "Description" "Buzzers Transducer, Externally Driven Piezo 3V 4kHz 60dB @ 3V, 10cm Through Hole PC Pins"
-			(at 647.7 15.24 0)
+			(at 632.46 43.18 0)
 			(hide yes)
 			(show_name no)
@@
 		)
 		(property "MF" "TDK"
-			(at 647.7 15.24 0)
+			(at 632.46 43.18 0)
 			(hide yes)
 			(show_name no)
@@
 		)
 		(property "MAXIMUM_PACKAGE_HEIGHT" "7.0mm"
-			(at 647.7 15.24 0)
+			(at 632.46 43.18 0)
 			(hide yes)
 			(show_name no)
@@
 		)
 		(property "PACKAGE" "SIP-5 TDK"
-			(at 647.7 15.24 0)
+			(at 632.46 43.18 0)
 			(hide yes)
 			(show_name no)
@@
 		)
 		(property "PRICE" "None"
-			(at 647.7 15.24 0)
+			(at 632.46 43.18 0)
 			(hide yes)
 			(show_name no)
@@
 		)
 		(property "MP" "PS1240P02CT3"
-			(at 647.7 15.24 0)
+			(at 632.46 43.18 0)
 			(hide yes)
 			(show_name no)
@@
 		)
 		(property "AVAILABILITY" "Unavailable"
-			(at 647.7 15.24 0)
+			(at 632.46 43.18 0)
 			(hide yes)
 			(show_name no)

Commit message: Schematic Updates
Parts:
- removed F1: 15 A, Resistor_THT:R_Axial_DIN0922_L20.0mm_D9.0mm_P25.40mm_Horizontal, symbol Device:Fuse
- removed L1, L2, L3: 3.3uH, Inductor_SMD:L_Eaton_SDCHA1V80, symbol Device:L
- added C86: 470 uF, Capacitor_THT:CP_Radial_D8.0mm_P3.80mm, symbol Device:C_Polarized
- added C87: 0.1uF, Capacitor_SMD:C_0603_1608Metric, symbol Device:C
- added D28, D29, D30, D31, D32, D33, D34, D35: D_Schottky, Diode_SMD:D_SMB, symbol Device:D_Schottky
- added D36, D37, D38, D39, D40, D41, D42: POWER, LED_SMD:LED_0603_1608Metric, symbol Device:LED
- added D43, D45, D47, D49, D51, D53: RXCAN, LED_SMD:LED_0603_1608Metric, symbol Device:LED
- added D44, D46, D48, D50, D52, D54: TXCAN, LED_SMD:LED_0603_1608Metric, symbol Device:LED
- added F2: 3557-2, 3557_2:FUSE_3557-2, symbol Device:3557-2
- added J16, J17: Conn_01x03_Pin, symbol Connector:Conn_01x03_Pin
- added JP2: SolderJumper_3_Bridged12, symbol Jumper:SolderJumper_3_Bridged12
- added L7, L8, L9: 4.7uH, Inductor_SMD:L_Eaton_SDCHA1V80, symbol Device:L
- added R78: 4K7, Resistor_SMD:R_0603_1608Metric, symbol Device:R_US
- added R79: 120, Resistor_SMD:R_0603_1608Metric, symbol Device:R_US
- added R80, R81, R82, R86: 1K, Resistor_SMD:R_0603_1608Metric, symbol Device:R_US
- added R83, R84, R85, R87, R88, R89, R90, R91, R92, R93, R94, R95, R96, R97, R98: 470, Resistor_SMD:R_0603_1608Metric, symbol Device:R_US
- added S5: TEST, SWT0210_045026GSA:SW_SWT0210-045026GSA_REVA, symbol Regulator_Switching:SWT0210-045026GSA_REVA
- added TP50, TP51, TP52, TP53, TP54, TP55: PG, TestPoint:TestPoint_Keystone_5015_Micro_Mini, symbol Connector:TestPoint
- R71: value 1ohm -> 200m; footprint Resistor_THT:R_Axial_Power_L48.0mm_W12.5mm_P60.96mm -> Resistor_THT:R_Axial_DIN0516_L15.5mm_D5.0mm_P25.40mm_Horizontal
- R74: now not fitted
- R75: footprint RES 330 OHM 1% 1/10W 0603 -> Resistor_SMD:R_0603_1608Metric
- TP29: value Z3_BOOT0 -> Z2_BOOT0
- TP30: value Z3_MCO -> Z2_MCO
Connections:
- net +12V: now also U20.4 (Vs), D32.1 (K), D33.1 (K), D34.1 (K), D35.1 (K), D42.2 (A), J16.1 (Pin_1), J17.1 (Pin_1); no longer U20.9 (Vss)
- net +3.3V_Z1: now also JP2.1 (A), R78.1; no longer JP25.2 (B)
- net +3.3V_Z2: now also FB2.1, JP31.2 (B), R69.1
- net +3.3V_Z3: no longer C62.1, C72.1, FB2.1, JP31.2 (B), R69.1, U3.1 (VBAT), U7.1 (VBAT)
- net +5V_Z3: now also U20.11 (EnB), U20.6 (EnA), U20.9 (Vss), C86.1; no longer U20.4 (Vs)
- net +7V_Z2: now also U5.3 (+)
- net ENC_LEFT_B: no longer J7.4 (Pin_4)
- net ENC_RIGHT_B: now also J7.4 (Pin_4)
- net GND: now also LS1.2, LS2.2, U20.1 (SENSE_A), C86.2, D28.2 (A), D29.2 (A), D30.2 (A), D31.2 (A), J16.3 (Pin_3), J17.3 (Pin_3), R79.2, R80.2, R81.2, R82.2, R83.2, R84.2, R85.2, R86.2, R87.2, R88.2, R89.2, R90.2, R91.2, R92.2, R93.2, R94.2, R95.2, R96.2, R97.2, R98.2, S5.3, S5.4
- net Z1_INT_CAN_A: now also J5.22 (GPIO25/SDIO_DAT1); no longer J5.18 (GPIO24/SDIO_DAT0)
- net Z1_INT_CAN_B: now also J5.18 (GPIO24/SDIO_DAT0); no longer J5.22 (GPIO25/SDIO_DAT1)
- net Z2_NRST: now also C70.2, S3.3, S3.4, U7.7 (NRST)
- net Z3_BOOT0: no longer R66.1, TP29.1, U7.60 (BOOT0)
- net Z3_NRST: no longer C70.2, S3.3, S3.4, U7.7 (NRST)
- net at C38.1, C39.1, C40.1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: now also D39.2 (A), L9.2
- net at C45.1, C46.1, C47.1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: now also D41.2 (A), L7.2
- net at D2.4 (DIN): now also U7.36 (PB15)
- net at C30.1, C31.1, C32.1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: now also D40.2 (A), L8.2
- net at D8.4 (DIN): now also U3.36 (PB15); no longer D7.2 (DOUT)
- net at Q2.2 (D): now also F2.2_1, F2.2_2
- net at J1.P (POS): now also F2.1_1, F2.1_2
- net at R71.2: now also J9.2 (Pin_2), U5.4 (-); no longer U5.3 (+)
- net at C59.1, C60.1, C61.1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: now also D38.2 (A)
- net at U1.1 (TXCAN), U8.1 (D): now also D44.2 (A)
- net at U1.2 (RXCAN), U8.4 (R): now also D43.2 (A)
- net at U11.1 (TXCAN), U12.1 (D): now also D52.2 (A)
- net at U11.2 (RXCAN), U12.4 (R): now also D51.2 (A)
- net at IC2.4 (PG), R41.1: now also TP54.1
- net at C52.1, C53.1, C54.1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: now also D36.2 (A)
- net at IC1.2 (SW): now also L8.1
- net at JP31.1 (A), U7.19 (VDD), U7.32 (VDD)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: now also C72.1, U7.1 (VBAT)
- net at U7.21 (PA5): now also LS1.1
- net at C83.1, C84.1, C85.1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: now also D37.2 (A)
- net at IC2.2 (SW): now also L9.1
- net at IC4.4 (PG), R53.1: now also TP51.1
- net at U17.1 (TXCAN), U18.1 (D): now also D54.2 (A)
- net at U17.2 (RXCAN), U18.4 (R): now also D53.2 (A)
- net at IC1.4 (PG), R10.1: now also TP53.1
- net at U20.2 (OUT1), U4.1 (IP+), U4.2 (IP+): now also D28.1 (K), D32.2 (A)
- net at IC5.4 (PG), R59.1: now also TP55.1
- net at IC3.2 (SW): now also L7.1
- net at U13.1 (TXCAN), U14.1 (D): now also D46.2 (A)
- net at U13.2 (RXCAN), U14.4 (R): now also D45.2 (A)
- net at IC3.4 (PG), R47.1: now also TP50.1
- net at JP30.1 (A), U3.19 (VDD), U3.32 (VDD)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: now also C62.1, U3.1 (VBAT)
- net at U15.1 (TXCAN), U16.1 (D): now also D48.2 (A)
- net at U15.2 (RXCAN), U16.4 (R): now also D47.2 (A)
- net at U3.21 (PA5): now also LS2.1
- net at J7.6 (Pin_6), U20.3 (OUT2): now also D29.1 (K), D33.2 (A)
- net at U10.1 (D), U9.1 (TXCAN): now also D50.2 (A)
- net at U10.4 (R), U9.2 (RXCAN): now also D49.2 (A)
- net at J8.1 (Pin_1), U20.13 (OUT3): now also D30.1 (K), D34.2 (A)
- net at U2.3 (IP-), U2.4 (IP-), U20.14 (OUT4): now also D31.1 (K), D35.2 (A)
- net PI_3.3V: now reaches J5.1 (3V3), J5.17 (3V3)
- net PI_3.3V: now also JP2.3 (B)
- net at J5.12 (GPIO18/SPI1_~{CE0}/PCM_CLK/PWM0): now also J16.2 (Pin_2)
- net at J5.38 (GPIO20/SPI1_MOSI/PCM_DIN/PWM1): now also J17.2 (Pin_2)
- net at IC6.4 (PG), R74.1: now also TP52.1
- new net: D37.1 (K), R81.1
- new net: D46.1 (K), R90.1
- new net: D52.1 (K), R96.1
- new net: D54.1 (K), R98.1
- new net: D45.1 (K), R89.1
- new net: D43.1 (K), R87.1
- new net: D53.1 (K), R97.1
- new net: D38.1 (K), R82.1
- new net: D39.1 (K), R83.1
- new net: D40.1 (K), R84.1
- new net: D48.1 (K), R92.1
- new net: D49.1 (K), R93.1
- new net: D51.1 (K), R95.1
- new net: D36.1 (K), R80.1
- new net: D44.1 (K), R88.1
- new net: C87.2, R79.1
- new net: D41.1 (K), R85.1
- new net: JP2.2 (C), JP25.2 (B)
- new net: D50.1 (K), R94.1
- new net: D42.1 (K), R86.1
- new net: D47.1 (K), R91.1
- new net Z1_TEST_BUTTON: C87.1, R78.2, S5.1, S5.2
- new net Z2_BOOT0: R66.1, TP29.1, U7.60 (BOOT0)
- no-connect marks 0 -> 75
Other:
- note removed: "Steering (Zone 2)"
- moved on the sheet: C25, C26, C63, C73, C74, C75, C76, C77, D19, D20, D23, J1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

Commit message: Updated pin definitions and NC to have 0 ERC errors. Still many warnings, most of which are footprint library related.
Connections:
- no-connect marks 75 -> 92

Commit message: made cleanup changes, put notes in doc
Connections:
- net GND: now also U20.15 (SENSE_B)
- no-connect marks 92 -> 91
Other:
- moved on the sheet: C25, C26, C74, C75, C76, C77, C86, D28, D29, D30, D31, D32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

Commit message: Small updates.
Parts:
- removed R37, R44, R50, R56, R62, R77: 53, Resistor_SMD:R_0603_1608Metric, symbol Device:R_US
Connections:
- net at C38.1, C39.1, C40.1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: now also C37.1, R42.2
- net at C45.1, C46.1, C47.1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: now also C44.1, R48.2
- net at C30.1, C31.1, C32.1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: now also C29.1, R22.2
- net at C59.1, C60.1, C61.1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: now also C58.1, R60.2
- net at C52.1, C53.1, C54.1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: now also C51.1, R54.2
- net at C83.1, C84.1, C85.1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: now also C82.1, R75.2

Commit message: Zone 2 complete
Parts:
- removed JP30: STM_POWER, Connector_PinHeader_2.54mm:PinHeader_1x02_P2.54mm_Vertical, symbol Jumper:Jumper_2_Bridged
- removed R67, R68, R8, R9: 0, Resistor_SMD:R_0603_1608Metric, symbol Device:R_US
- removed TP32: Z3_ERR, TestPoint:TestPoint_Keystone_5015_Micro_Mini, symbol Connector:TestPoint
- removed TP33: Z1_CANL_A, TestPoint:TestPoint_Keystone_5015_Micro_Mini, symbol Connector:TestPoint
- removed TP34: Z1_CANH_A, TestPoint:TestPoint_Keystone_5015_Micro_Mini, symbol Connector:TestPoint
- removed TP35: Z1_CANH_B, TestPoint:TestPoint_Keystone_5015_Micro_Mini, symbol Connector:TestPoint
- removed TP36: Z1_CANL_B, TestPoint:TestPoint_Keystone_5015_Micro_Mini, symbol Connector:TestPoint
- removed TP37: Z2_CANH_B, TestPoint:TestPoint_Keystone_5015_Micro_Mini, symbol Connector:TestPoint
- removed TP38: Z2_CANL_B, TestPoint:TestPoint_Keystone_5015_Micro_Mini, symbol Connector:TestPoint
- removed TP39: Z2_CANH_A, TestPoint:TestPoint_Keystone_5015_Micro_Mini, symbol Connector:TestPoint
- removed TP40: Z2_CANL_A, TestPoint:TestPoint_Keystone_5015_Micro_Mini, symbol Connector:TestPoint
- removed TP41: Z3_CANH_B, TestPoint:TestPoint_Keystone_5015_Micro_Mini, symbol Connector:TestPoint
- removed TP42: Z3_CANL_B, TestPoint:TestPoint_Keystone_5015_Micro_Mini, symbol Connector:TestPoint
- removed TP43: Z3_CANH_A, TestPoint:TestPoint_Keystone_5015_Micro_Mini, symbol Connector:TestPoint
- removed TP44: Z3_CANL_A, TestPoint:TestPoint_Keystone_5015_Micro_Mini, symbol Connector:TestPoint
- added C100, C88, C89, C90, C91, C92, C93, C94, C95, C96, C98: 0.1uF, Capacitor_SMD:C_0603_1608Metric, symbol Device:C
- added C97, C99: 1uF, Capacitor_SMD:C_0603_1608Metric, symbol Device:C
- added JP34: STM_POWER, Connector_PinHeader_2.54mm:PinHeader_1x02_P2.54mm_Vertical, symbol Jumper:Jumper_2_Bridged
- added R44, R50, R56, R62: 10k, Resistor_SMD:R_0603_1608Metric, symbol Device:R_US
- added R77: 120, Resistor_SMD:R_0603_1608Metric, symbol Device:R_US
- added TP56, TP57, TP58, TP76, TP77, TP78, TP79: GND, TestPoint:TestPoint_Keystone_5015_Micro_Mini, symbol Connector:TestPoint
- added TP59: DIR_A, TestPoint:TestPoint_Keystone_5015_Micro_Mini, symbol Connector:TestPoint
- added TP60: MOTOR_LEFT_PWM, TestPoint:TestPoint_Keystone_5015_Micro_Mini, symbol Connector:TestPoint
- added TP61, TP71, TP74: ERR, TestPoint:TestPoint_Keystone_5015_Micro_Mini, symbol Connector:TestPoint
- added TP62: SERVO_PWM, TestPoint:TestPoint_Keystone_5015_Micro_Mini, symbol Connector:TestPoint
- added TP63: RR, TestPoint:TestPoint_Keystone_5015_Micro_Mini, symbol Connector:TestPoint
- added TP64: RL, TestPoint:TestPoint_Keystone_5015_Micro_Mini, symbol Connector:TestPoint
- added TP65, TP68, TP73: DEG_B, TestPoint:TestPoint_Keystone_5015_Micro_Mini, symbol Connector:TestPoint
- added TP66, TP67, TP72: DEG_A, TestPoint:TestPoint_Keystone_5015_Micro_Mini, symbol Connector:TestPoint
- added TP69: FL, TestPoint:TestPoint_Keystone_5015_Micro_Mini, symbol Connector:TestPoint
- added TP70: FR, TestPoint:TestPoint_Keystone_5015_Micro_Mini, symbol Connector:TestPoint
- added TP75: CUR_POST, TestPoint:TestPoint_Keystone_5015_Micro_Mini, symbol Connector:TestPoint
- C62: value 1uF -> 0.1uF
- C74: value 0.1uF -> 1uF
- D10, D15, D20: value DEGRADED -> DEGRADED_B
- D14, D19, D9: value DEGRADED -> DEGRADED_A
- FB1, FB2: footprint Inductor_SMD:L_0201_0603Metric -> Inductor_SMD:L_0603_1608Metric
- J16, J17: footprint (none) -> Connector_PinHeader_2.54mm:PinHeader_1x03_P2.54mm_Vertical
- JP1, JP11, JP19, JP9: value (none) -> TERM
- JP2: value SolderJumper_3_Bridged12 -> 3.3 Souce; footprint (none) -> Jumper:SolderJumper-3_P1.3mm_Bridged12_RoundedPad1.0x1.5mm_NumberLabels
- R75: value 91K -> 510K
- R76: value 10K -> 47K
- TP101: renamed from Z2_CAN_TX_A1; value CMD_TX -> Z2_CAN_TX_A
- TP15: value MOTOR_PWM_OUT -> MOTOR_RIGHT_PWM
- TP47: value SERVO_CURRENT -> CURR_PRE
- TP48: value Z3_5_EN -> Z2_5_EN
- TP8: value Z2_CAN_RX_B -> Z2_CAN_TX_B
Connections:
- net +3.3V_Z1: now also JP2.2 (C); no longer JP2.1 (A)
- net +3.3V_Z3: now also JP34.2 (B)
- net +5V_Z1: no longer D2.1 (VDD), D3.1 (VDD), D4.1 (VDD), D5.1 (VDD), D6.1 (VDD), D7.1 (VDD)
- net +5V_Z3: now also C88.1, C89.1
- net +7V_Z2: now also D2.1 (VDD), D3.1 (VDD), D4.1 (VDD), D5.1 (VDD), D6.1 (VDD), D7.1 (VDD)
- net DIR_A: now also TP59.1
- net FL_BLINK: now also TP69.1
- net FR_BLINK: now also TP70.1
- net GND: now also C100.2, C88.2, C89.2, C90.2, C91.2, C92.2, C93.2, C94.2, C95.2, C96.2, C97.2, C98.2, C99.2, R44.2, R50.2, R56.2, R62.2, TP56.1, TP57.1, TP58.1, TP76.1, TP77.1, TP78.1, TP79.1
- net MOTOR_CURRENT_LEFT: no longer C74.1
- net MOTOR_CURRENT_RIGHT: no longer C77.1
- net MOTOR_LEFT_DIR: now also R44.1
- net MOTOR_LEFT_PWM: now also R50.1, TP60.1
- net MOTOR_RIGHT_DIR: now also R56.1
- net MOTOR_RIGHT_PWM: now also R62.1
- net RL_BLINK: now also TP64.1
- net RR_BLINK: now also TP63.1
- net SERVO_CURRENT: now also C100.1, R77.2, TP75.1; no longer TP47.1, U5.1
- net SERVO_PWM: now also TP62.1
- net Z1_DEG_A: now also TP72.1
- net Z1_DEG_B: now also TP73.1
- net Z1_ERR: now also TP74.1
- net Z1_TEST_BUTTON: now also J5.27 (ID_SD_I2C0/GPIO00)
- net Z2_DEG_A: now also TP67.1
- net Z2_DEG_B: now also TP68.1
- net Z2_ERR: now also TP71.1
- net Z2_SCLK: now also U7.21 (PA5); no longer J3.6 (Pin_6), U7.55 (PB3)
- net Z3_DEG_A: now also TP66.1
- net Z3_DEG_B: now also TP65.1
- net Z3_ERR: now also TP61.1
- net Z3_SCLK: now also U3.21 (PA5); no longer J2.6 (Pin_6), U3.55 (PB3)
- net at C68.2, Y8.1: now also U7.3 (PC14)
- net at C66.1, Y7.4: now also U3.4 (PC15)
- net at C69.1, Y8.4: now also U7.4 (PC15)
- net STM_POWER_Z2: now reaches C72.1, JP31.1 (A), U7.1 (VBAT), U7.19 (VDD), U7.32 (VDD), U7.48 (VDD), U7.64 (VDD)
- net STM_POWER_Z2: now also C92.1, C93.1, C94.1, C95.1
- net at FB2.2, U7.13 (VREF+): now also C96.1, C97.1
- net at LS1.1: now also U7.50 (PA15); no longer U7.21 (PA5)
- net at FB1.2, U3.13 (VREF+): now also C98.1, C99.1
- net at C65.2, Y7.1: now also U3.3 (PC14)
- net STM_POWER_Z3: now reaches C62.1, U3.1 (VBAT), U3.19 (VDD), U3.32 (VDD), U3.48 (VDD), U3.64 (VDD)
- net STM_POWER_Z3: now also C74.1, C77.1, C90.1, C91.1, JP34.1 (A)
- net at JP25.2 (B): now also JP2.1 (A); no longer JP2.2 (C)
- net at LS2.1: now also U3.50 (PA15); no longer U3.21 (PA5)
- new net: R77.1, TP47.1, U5.1
- new net Z2_SWO: J3.6 (Pin_6), U7.55 (PB3)
- new net Z3_SWO: J2.6 (Pin_6), U3.55 (PB3)
- no-connect marks 91 -> 89
Other:
- note removed: "Notes: - AGND and GND are shared - This layout doens't have pin 31 or 47, but they should be tied to ground and that seems correct on the PCB. They are potentially suppsoed to have a 2.2 uF cap - The 8Mhz oscillator is not connected"
- moved on the sheet: C25, C26, C63, C64, C65, C66, C67, C73, C75, C76, C86, D10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

Commit message: Most of Z3 routed.
Parts:
- added JP3: SolderJumper_2_Bridged, Jumper:SolderJumper-2_P1.3mm_Bridged_RoundedPad1.0x1.5mm, symbol Jumper:SolderJumper_2_Bridged
Connections:
- net +7V_Z2: now also JP3.2 (B); no longer D2.1 (VDD), D3.1 (VDD), D4.1 (VDD), D5.1 (VDD), D6.1 (VDD), D7.1 (VDD)
- net CANH_B: now also R21.1; no longer JP19.1 (A)
- net CANL_B: now also JP19.1 (A); no longer R21.2
- net MOTOR_CURRENT_LEFT: now also U3.24 (PC4); no longer U3.11 (PC3)
- net MOTOR_CURRENT_RIGHT: now also U3.11 (PC3); no longer U3.24 (PC4)
- net MOTOR_PWR-_L: now reaches D30.1 (K), D34.2 (A), J8.1 (Pin_1), U20.13 (OUT3)
- net MOTOR_PWR-_R: now reaches D29.1 (K), D33.2 (A), J7.6 (Pin_6), U20.3 (OUT2)
- net MOTOR_PWR+_L: now reaches D31.1 (K), D35.2 (A), U2.3 (IP-), U2.4 (IP-), U20.14 (OUT4)
- net MOTOR_PWR+_R: now reaches D28.1 (K), D32.2 (A), U20.2 (OUT1), U4.1 (IP+), U4.2 (IP+)
- net MOTOR_PWR+C_R: now reaches J7.1 (Pin_1), U4.3 (IP-), U4.4 (IP-)
- net at JP19.2 (B): now also R21.2; no longer R21.1
- net MOTOR_PWR+C_L: now reaches J8.6 (Pin_6), U2.1 (IP+), U2.2 (IP+)
- new net: D2.1 (VDD), D3.1 (VDD), D4.1 (VDD), D5.1 (VDD), D6.1 (VDD), D7.1 (VDD), JP3.1 (A)
Other:
- moved on the sheet: JP19

Commit message: Initial Board layout complete and DRC passes
Parts:
- removed TP31: Z3_ERR, TestPoint:TestPoint_Keystone_5015_Micro_Mini, symbol Connector:TestPoint
- added JP4: SolderJumper_2_Bridged, Jumper:SolderJumper-2_P1.3mm_Bridged_RoundedPad1.0x1.5mm, symbol Jumper:SolderJumper_2_Bridged
- added TP80, TP81, TP82, TP83: GND, TestPoint:TestPoint_Keystone_5015_Micro_Mini, symbol Connector:TestPoint
- JP3: value SolderJumper_2_Bridged -> PIXEL POWER
- TP16: value Z3_CAN_TX_A -> CAN_TX_A
- TP18: value Z3_CAN_RX_A -> CAN_RX_A
- TP19: value Z3_CAN_RX_B -> CAN_RX_B
Connections:
- net +5V_Z1: no longer D21.1 (VDD), D22.1 (VDD), D24.1 (VDD), D25.1 (VDD), D26.1 (VDD), D27.1 (VDD), D8.1 (VDD)
- net +5V_Z3: now also JP4.2 (B)
- net GND: now also TP80.1, TP81.1, TP82.1, TP83.1
- new net: D21.1 (VDD), D22.1 (VDD), D24.1 (VDD), D25.1 (VDD), D26.1 (VDD), D27.1 (VDD), D8.1 (VDD), JP4.1 (A)
